File: hardware/klein_star_ein/klein_star_ein.kicad_sch (KiCad schematic)
At the start: 0 parts

Commit message: fixed DRAM, added initial schematic
Parts:
- added C1, C10, C11, C12, C14, C15, C17, C18, C19, C2, C20, C3, C4, C5, C7, C9: 0.1uF, Capacitor_SMD:C_0402_1005Metric, symbol Device:C_Small
- added C13, C16, C6, C8: 4.7uF, Capacitor_SMD:C_0402_1005Metric, symbol Device:C_Small
- added R1, R2, R7, R8: 51R, Resistor_SMD:R_0402_1005Metric, symbol Device:R_Small
- added R3, R5: 240R, Resistor_SMD:R_0402_1005Metric, symbol Device:R_Small
- added R4, R6: 0R, Resistor_SMD:R_1206_3216Metric_Pad1.30x1.75mm_HandSolder, symbol Device:R_Small
- added U1: ECP5UM25, Package_BGA:Lattice_caBGA-381_17.0x17.0mm_Layout20x20_P0.8mm_Ball0.4mm_Pad0.4mm_NSMD, symbol ECP5UM25:ECP5UM25
- added U2, U3: MT41K512M16, Package_BGA:BGA-96_9.0x13.0mm_Layout2x3x16_P0.8mm, symbol MT41K512M16:MT41K512M16
Connections:
- new net: C4.1, R1.2, R2.2
- new net: R5.1, U3.L8 (ZQ)
- new net: C20.1, R7.2, R8.2
- new net: R3.1, U2.L8 (ZQ)
- new net BANK_AH_RDQS: U1.E4 (PL8A/LDQS8/-), U3.C7 (UDQS)
- new net BANK_AH_RDQSN: U1.D5 (PL8B/LDQSN8/-), U3.B7 (UDQS#)
- new net BANK_AL_RDQS: U1.H4 (PL20A/LDQS20/GR_PCLK7_1), U3.F3 (LDQS)
- new net BANK_AL_RDQSN: U1.G5 (PL20B/LDQSN20/-), U3.G3 (LDQS#)
- new net BANK_A_DQ0: U1.A2 (PL14A/LDQ20/-), U3.E3 (DQ0)
- new net BANK_A_DQ1: U1.B1 (PL14B/LDQ20/-), U3.F7 (DQ1)
- new net BANK_A_DQ10: U1.A3 (PL5C/LDQ8/-), U3.C8 (DQ10)
- new net BANK_A_DQ11: U1.B3 (PL5D/LDQ8/-), U3.C2 (DQ11)
- new net BANK_A_DQ12: U1.F4 (PL11A/LDQ8/-), U3.A7 (DQ12)
- new net BANK_A_DQ13: U1.E3 (PL11B/LDQ8/-), U3.A2 (DQ13)
- new net BANK_A_DQ14: U1.E5 (PL11C/LDQ8/-), U3.B8 (DQ14)
- new net BANK_A_DQ15: U1.F5 (PL11D/LDQ8/-), U3.A3 (DQ15)
- new net BANK_A_DQ2: U1.C1 (PL17A/LDQ20/-), U3.F2 (DQ2)
- new net BANK_A_DQ3: U1.D1 (PL17B/LDQ20/-), U3.F8 (DQ3)
- new net BANK_A_DQ4: U1.G3 (PL23A/LDQ20/PCLKT7_1), U3.H3 (DQ4)
- new net BANK_A_DQ5: U1.F3 (PL23B/LDQ20/PCLKC7_1), U3.H8 (DQ5)
- new net BANK_A_DQ6: U1.F2 (PL23C/LDQ20/PCLKT7_0), U3.G2 (DQ6)
- new net BANK_A_DQ7: U1.E2 (PL23D/LDQ20/PCLKC7_0), U3.H7 (DQ7)
- new net BANK_A_DQ8: U1.C4 (PL5A/LDQ8/-), U3.D7 (DQ8)
- new net BANK_A_DQ9: U1.B4 (PL5B/LDQ8/-), U3.C3 (DQ9)
- new net BANK_A_VREF: U1.B2 (PL14C/LDQ20/VREF1_7)
- new net BANK_BH_RDQS: U1.F17 (PR8A/RDQS8/-), U2.C7 (UDQS)
- new net BANK_BH_RDQSN: U1.G18 (PR8B/RDQSN8/-), U2.B7 (UDQS#)
- new net BANK_BL_RDQS: U1.G19 (PR20A/RDQS20/GR_PCLK2_1), U2.F3 (LDQS)
- new net BANK_BL_RDQSN: U1.H20 (PR20B/RDQSN20/-), U2.G3 (LDQS#)
- new net BANK_B_DQ0: U1.C20 (PR14A/RDQ20/-), U2.E3 (DQ0)
- new net BANK_B_DQ1: U1.D19 (PR14B/RDQ20/-), U2.F7 (DQ1)
- new net BANK_B_DQ10: U1.E18 (PR5C/RDQ8/-), U2.C8 (DQ10)
- new net BANK_B_DQ11: U1.F18 (PR5D/RDQ8/-), U2.C2 (DQ11)
- new net BANK_B_DQ12: U1.H18 (PR11A/RDQ8/-), U2.A7 (DQ12)
- new net BANK_B_DQ13: U1.H17 (PR11B/RDQ8/-), U2.A2 (DQ13)
- new net BANK_B_DQ14: U1.J17 (PR11C/RDQ8/-), U2.B8 (DQ14)
- new net BANK_B_DQ15: U1.J16 (PR11D/RDQ8/-), U2.A3 (DQ15)
- new net BANK_B_DQ2: U1.E20 (PR17A/RDQ20/-), U2.F2 (DQ2)
- new net BANK_B_DQ3: U1.F19 (PR17B/RDQ20/-), U2.F8 (DQ3)
- new net BANK_B_DQ4: U1.J19 (PR23A/RDQ20/PCLKT2_1), U2.H3 (DQ4)
- new net BANK_B_DQ5: U1.K19 (PR23B/RDQ20/PCLKC2_1), U2.H8 (DQ5)
- new net BANK_B_DQ6: U1.J20 (PR23C/RDQ20/PCLKT2_0), U2.G2 (DQ6)
- new net BANK_B_DQ7: U1.K20 (PR23D/RDQ20/PCLKC2_0), U2.H7 (DQ7)
- new net BANK_B_DQ8: U1.D18 (PR5A/RDQ8/-), U2.D7 (DQ8)
- new net BANK_B_DQ9: U1.E17 (PR5B/RDQ8/-), U2.C3 (DQ9)
- new net BANK_B_VREF: U1.D20 (PR14C/RDQ20/VREF1_2)
- new net DRAMREF: C1.1, C11.1, C14.1, C17.1, C2.1, C3.1, U2.H1 (Vrefdq), U2.M8 (Vrefca), U3.H1 (Vrefdq), U3.M8 (Vrefca)
- new net DRAM_ADDR_0: U2.N3 (A0), U3.N3 (A0)
- new net DRAM_ADDR_1: U2.P7 (A1), U3.P7 (A1)
- new net DRAM_ADDR_10: U2.L7 (A10), U3.L7 (A10)
- new net DRAM_ADDR_11: U2.R7 (A11), U3.R7 (A11)
- new net DRAM_ADDR_12: U2.N7 (A12), U3.N7 (A12)
- new net DRAM_ADDR_13: U2.T3 (A13), U3.T3 (A13)
- new net DRAM_ADDR_14: U2.T7 (A14), U3.T7 (A14)
- new net DRAM_ADDR_15: U2.M7 (A15), U3.M7 (A15)
- new net DRAM_ADDR_2: U2.P3 (A2), U3.P3 (A2)
- new net DRAM_ADDR_3: U2.N2 (A3), U3.N2 (A3)
- new net DRAM_ADDR_4: U2.P8 (A4), U3.P8 (A4)
- new net DRAM_ADDR_5: U2.P2 (A5), U3.P2 (A5)
- new net DRAM_ADDR_6: U2.R8 (A6), U3.R8 (A6)
- new net DRAM_ADDR_7: U2.R2 (A7), U3.R2 (A7)
- new net DRAM_ADDR_8: U2.T8 (A8), U3.T8 (A8)
- new net DRAM_ADDR_9: U2.R3 (A9), U3.R3 (A9)
- new net DRAM_ADDR_BA0: U2.M2 (BA0), U3.M2 (BA0)
- new net DRAM_ADDR_BA1: U2.N8 (BA1), U3.N8 (BA1)
- new net DRAM_ADDR_BA2: U2.M3 (BA2), U3.M3 (BA2)
- new net DRAM_A_CKE: U1.C3 (PL8C/LDQ8/-), U3.K9 (CKE)
- new net DRAM_A_CK_N: R8.1, U1.A4 (PL2A/LDQ8/-), U3.K7 (CK#)
- new net DRAM_A_CK_P: R7.1, U1.A5 (PL2B/LDQ8/-), U3.J7 (CK)
- new net DRAM_A_LDM: U1.H3 (PL20D/LDQ20/-), U3.E7 (LDM)
- new net DRAM_A_ODT: U1.D3 (PL8D/LDQ8/-), U3.K1 (ODT)
- new net DRAM_A_UDM: U1.H5 (PL20C/LDQ20/GR_PCLK7_0), U3.D3 (UDM)
- new net DRAM_A_nCAS: U1.B5 (PL2C/LDQ8/-), U3.K3 (CAS#)
- new net DRAM_A_nCS: U1.D2 (PL17C/LDQ20/-), U3.L2 (CS#)
- new net DRAM_A_nRAS: U1.C5 (PL2D/LDQ8/-), U3.J3 (RAS#)
- new net DRAM_A_nRESET: U1.C2 (PL14D/LDQ20/-), U3.T2 (RESET#)
- new net DRAM_A_nWE: U1.E1 (PL17D/LDQ20/-), U3.L3 (WE#)
- new net DRAM_B_CKE: U1.G16 (PR8C/RDQ8/-), U2.K9 (CKE)
- new net DRAM_B_CK_N: R2.1, U1.C18 (PR2A/RDQ8/-), U2.K7 (CK#)
- new net DRAM_B_CK_P: R1.1, U1.D17 (PR2B/RDQ8/S0_IN), U2.J7 (CK)
- new net DRAM_B_LDM: U1.K18 (PR20D/RDQ20/-), U2.E7 (LDM)
- new net DRAM_B_ODT: U1.H16 (PR8D/RDQ8/-), U2.K1 (ODT)
- new net DRAM_B_UDM: U1.J18 (PR20C/RDQ20/GR_PCLK2_0), U2.D3 (UDM)
- new net DRAM_B_nCAS: U1.E16 (PR2C/RDQ8/-), U2.K3 (CAS#)
- new net DRAM_B_nCS: U1.F20 (PR17C/RDQ20/-), U2.L2 (CS#)
- new net DRAM_B_nRAS: U1.F16 (PR2D/RDQ8/-), U2.J3 (RAS#)
- new net DRAM_B_nRESET: U1.E19 (PR14D/RDQ20/-), U2.T2 (RESET#)
- new net DRAM_B_nWE: U1.G20 (PR17D/RDQ20/-), U2.L3 (WE#)
- new net DRAM_SUPPLY_A: C12.1, C13.1, C15.1, C16.1, C18.1, C19.1, R6.2, U3.A1 (Vddq), U3.A8 (Vddq), U3.B2 (Vdd), U3.C1 (Vddq), U3.C9 (Vddq), U3.D2 (Vddq), U3.D9 (Vdd), U3.E9 (Vddq), U3.F1 (Vddq), U3.G7 (Vdd), U3.H2 (Vddq), U3.H9 (Vddq), U3.K2 (Vdd), U3.K8 (Vdd), U3.N1 (Vdd), U3.N9 (Vdd), U3.R1 (Vdd), U3.R9 (Vdd)
- new net DRAM_SUPPLY_B: C10.1, C5.1, C6.1, C7.1, C8.1, C9.1, R4.2, U2.A1 (Vddq), U2.A8 (Vddq), U2.B2 (Vdd), U2.C1 (Vddq), U2.C9 (Vddq), U2.D2 (Vddq), U2.D9 (Vdd), U2.E9 (Vddq), U2.F1 (Vddq), U2.G7 (Vdd), U2.H2 (Vddq), U2.H9 (Vddq), U2.K2 (Vdd), U2.K8 (Vdd), U2.N1 (Vdd), U2.N9 (Vdd), U2.R1 (Vdd), U2.R9 (Vdd)
- new net DRAM_SUPPLY_GLOB: R4.1, R6.1, U1.H14 (VCCIO2/-), U1.H15 (VCCIO2/-), U1.J15 (VCCIO2/-)
- new net GND: C1.2, C10.2, C11.2, C12.2, C13.2, C14.2, C15.2, C16.2, C17.2, C18.2, C19.2, C2.2, C20.2, C3.2, C4.2, C5.2, C6.2, C7.2, C8.2, C9.2, R3.2, R5.2, U1.B14 (GND/-), U1.B7 (GND/-), U1.C19 (GND/-), U1.D4 (GND/-), U1.F13 (GND/-), U1.F14 (GND/-), U1.F7 (GND/-), U1.F8 (GND/-), U1.G10 (GND/-), U1.G11 (GND/-), U1.G12 (GND/-), U1.G13 (GND/-), U1.G14 (GND/-), U1.G15 (GND/-), U1.G17 (GND/-), U1.G4 (GND/-), U1.G6 (GND/-), U1.G7 (GND/-), U1.G8 (GND/-), U1.G9 (GND/-), U1.H19 (GND/-), U1.J10 (GND/-), U1.J11 (GND/-), U1.J12 (GND/-), U1.J14 (GND/-), U1.J2 (GND/-), U1.J7 (GND/-), U1.J9 (GND/-), U1.K10 (GND/-), U1.K11 (GND/-), U1.K12 (GND/-), U1.K14 (GND/-), U1.K15 (GND/-), U1.K6 (GND/-), U1.K7 (GND/-), U1.K9 (GND/-), U1.L10 (GND/-), U1.L11 (GND/-), U1.L12 (GND/-), U1.L9 (GND/-), U1.M10 (GND/-), U1.M11 (GND/-), U1.M12 (GND/-), U1.M14 (GND/-), U1.M16 (GND/-), U1.M2 (GND/-), U1.M7 (GND/-), U1.M9 (GND/-), U1.N14 (GND/-), U1.N15 (GND/-), U1.N6 (GND/-), U1.N7 (GND/-), U1.P11 (GND/-), U1.P12 (GND/-), U1.P13 (GND/-), U1.P14 (GND/-), U1.P7 (GND/-), U1.P8 (GND/-), U1.R19 (GND/-), U1.U10 (GND/GND), U1.U11 (GND/GND), U1.U12 (GND/GND), U1.U13 (GND/GND), U1.U14 (GND/GND), U1.U7 (GND/GND), U1.U8 (GND/GND), U1.U9 (GND/GND), U1.V12 (GND/GND), U1.V13 (GND/GND), U1.V14 (GND/GND), U1.V15 (GND/GND), U1.V16 (GND/GND), U1.V19 (GND/GND), U1.V20 (GND/GND), U1.V5 (GND/GND), U1.V6 (GND/GND), U1.V7 (GND/GND), U1.V8 (GND/GND), U1.V9 (GND/GND), U1.W12 (GND/GND), U1.W15 (GND/GND), U1.W16 (GND/GND), U1.W19 (GND/GND), U1.W6 (GND/GND), U1.W7 (GND/GND), U2.A9 (Vss), U2.B1 (Vssq), U2.B3 (Vss), U2.B9 (Vssq), U2.D1 (Vssq), U2.D8 (Vssq), U2.E1 (Vss), U2.E2 (Vssq), U2.E8 (Vssq), U2.F9 (Vssq), U2.G1 (Vssq), U2.G8 (Vss), U2.G9 (Vssq), U2.J2 (Vss), U2.J8 (Vss), U2.M1 (Vss), U2.M9 (Vss), U2.P1 (Vss), U2.P9 (Vss), U2.T1 (Vss), U2.T9 (Vss), U3.A9 (Vss), U3.B1 (Vssq), U3.B3 (Vss), U3.B9 (Vssq), U3.D1 (Vssq), U3.D8 (Vssq), U3.E1 (Vss), U3.E2 (Vssq), U3.E8 (Vssq), U3.F9 (Vssq), U3.G1 (Vssq), U3.G8 (Vss), U3.G9 (Vssq), U3.J2 (Vss), U3.J8 (Vss), U3.M1 (Vss), U3.M9 (Vss), U3.P1 (Vss), U3.P9 (Vss), U3.T1 (Vss), U3.T9 (Vss)
- no-connect marks 0 -> 26
Other:
- note added: "DRAM A SUPPLY"
- note added: "DRAM B SUPPLY"
