File: hardware/klein_star_ein/klein_star_ein.kicad_sch (KiCad schematic)
At the start: 31 parts, among them U1 ECP5UM25, U2 MT41K512M16, U3 MT41K512M16

Commit message: no idea what's here
Connections:
- net at U1.A10 (PT27A/PCLKT0_1): now also U1.A11 (PT27B/PCLKC0_1), U1.A6 (PT4A/-), U1.A7 (PT18A/-), U1.A8 (PT18B/-), U1.A9 (PT24A/GR_PCLK0_1), U1.B10 (PT24B/GR_PCLK0_0), U1.B11 (PT29A/PCLKT0_0), U1.B6 (PT4B/-), U1.B8 (PT15B/-), U1.B9 (PT22A/-), U1.C10 (PT22B/-), U1.C11 (PT29B/PCLKC0_0), U1.C6 (PT11A/-), U1.C7 (PT11B/-), U1.C8 (PT15A/-), U1.D6 (PT6B/-), U1.D7 (PT9B/-), U1.D8 (PT13B/-), U1.D9 (PT20A/-), U1.E6 (PT6A/-), U1.E7 (PT9A/-), U1.E8 (PT13A/-), U1.E9 (PT20B/-)
Other:
- moved on the sheet: U1A
Changed lines of the file:
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@@
 (kicad_sch (version 20201015) (generator eeschema)
   (paper "A0")
+  (junction (at 648.97 266.7) (diameter 0.9144) (color 0 0 0 0))
+  (junction (at 648.97 271.78) (diameter 0.9144) (color 0 0 0 0))
+  (junction (at 648.97 274.32) (diameter 0.9144) (color 0 0 0 0))
+  (junction (at 648.97 279.4) (diameter 0.9144) (color 0 0 0 0))
+  (junction (at 648.97 281.94) (diameter 0.9144) (color 0 0 0 0))
+  (junction (at 648.97 287.02) (diameter 0.9144) (color 0 0 0 0))
+  (junction (at 648.97 289.56) (diameter 0.9144) (color 0 0 0 0))
+  (junction (at 648.97 294.64) (diameter 0.9144) (color 0 0 0 0))
+  (junction (at 648.97 297.18) (diameter 0.9144) (color 0 0 0 0))
+  (junction (at 648.97 302.26) (diameter 0.9144) (color 0 0 0 0))
+  (junction (at 648.97 304.8) (diameter 0.9144) (color 0 0 0 0))
+  (junction (at 648.97 309.88) (diameter 0.9144) (color 0 0 0 0))
+  (junction (at 648.97 312.42) (diameter 0.9144) (color 0 0 0 0))
+  (junction (at 648.97 317.5) (diameter 0.9144) (color 0 0 0 0))
+  (junction (at 648.97 320.04) (diameter 0.9144) (color 0 0 0 0))
+  (junction (at 648.97 325.12) (diameter 0.9144) (color 0 0 0 0))
+  (junction (at 648.97 327.66) (diameter 0.9144) (color 0 0 0 0))
+  (junction (at 648.97 332.74) (diameter 0.9144) (color 0 0 0 0))
+  (junction (at 648.97 335.28) (diameter 0.9144) (color 0 0 0 0))
+  (junction (at 648.97 340.36) (diameter 0.9144) (color 0 0 0 0))
+  (junction (at 648.97 342.9) (diameter 0.9144) (color 0 0 0 0))
+  (junction (at 648.97 347.98) (diameter 0.9144) (color 0 0 0 0))
   (junction (at 833.12 161.29) (diameter 0.9144) (color 0 0 0 0))
   (junction (at 833.12 163.83) (diameter 0.9144) (color 0 0 0 0))
@@
   (junction (at 1161.415 77.47) (diameter 0.9144) (color 0 0 0 0))
   (junction (at 1162.685 151.765) (diameter 0.9144) (color 0 0 0 0))
-  (no_connect (at 1066.8 572.77))
+  (no_connect (at 1066.8 570.23))
+  (no_connect (at 1066.8 539.75))
+  (no_connect (at 1066.8 560.07))
+  (no_connect (at 1066.8 529.59))
+  (no_connect (at 1066.8 519.43))
+  (no_connect (at 1066.8 527.05))
+  (no_connect (at 1066.8 542.29))
+  (no_connect (at 1066.8 532.13))
+  (no_connect (at 1066.8 575.31))
+  (no_connect (at 1066.8 521.97))
   (no_connect (at 1066.8 544.83))
+  (no_connect (at 1066.8 562.61))
+  (no_connect (at 1066.8 549.91))
+  (no_connect (at 1066.8 557.53))
+  (no_connect (at 1066.8 582.93))
+  (no_connect (at 1066.8 577.85))
   (no_connect (at 1066.8 565.15))
   (no_connect (at 1066.8 524.51))
-  (no_connect (at 1066.8 577.85))
-  (no_connect (at 1066.8 560.07))
-  (no_connect (at 1066.8 562.61))
-  (no_connect (at 1066.8 542.29))
-  (no_connect (at 1066.8 570.23))
-  (no_connect (at 1066.8 529.59))
+  (no_connect (at 1066.8 554.99))
   (no_connect (at 1066.8 567.69))
-  (no_connect (at 1066.8 532.13))
-  (no_connect (at 1066.8 549.91))
-  (no_connect (at 1066.8 519.43))
+  (no_connect (at 1066.8 547.37))
+  (no_connect (at 1066.8 534.67))
   (no_connect (at 1066.8 537.21))
   (no_connect (at 1066.8 552.45))
-  (no_connect (at 1066.8 557.53))
-  (no_connect (at 1066.8 534.67))
-  (no_connect (at 1066.8 575.31))
-  (no_connect (at 1066.8 521.97))
+  (no_connect (at 1066.8 572.77))
   (no_connect (at 1066.8 580.39))
-  (no_connect (at 1066.8 554.99))
-  (no_connect (at 1066.8 582.93))
-  (no_connect (at 1066.8 547.37))
-  (no_connect (at 1066.8 539.75))
-  (no_connect (at 1066.8 527.05))
+  (wire (pts (xy 648.97 264.16) (xy 648.97 266.7))
+    (stroke (width 0) (type solid) (color 0 0 0 0))
+  )
+  (wire (pts (xy 648.97 266.7) (xy 648.97 271.78))
+    (stroke (width 0) (type solid) (color 0 0 0 0))
+  )
+  (wire (pts (xy 648.97 271.78) (xy 648.97 274.32))
+    (stroke (width 0) (type solid) (color 0 0 0 0))
+  )
+  (wire (pts (xy 648.97 274.32) (xy 648.97 279.4))
+    (stroke (width 0) (type solid) (color 0 0 0 0))
+  )
+  (wire (pts (xy 648.97 279.4) (xy 648.97 281.94))
+    (stroke (width 0) (type solid) (color 0 0 0 0))
+  )
+  (wire (pts (xy 648.97 281.94) (xy 648.97 287.02))
+    (stroke (width 0) (type solid) (color 0 0 0 0))
+  )
+  (wire (pts (xy 648.97 287.02) (xy 648.97 289.56))
+    (stroke (width 0) (type solid) (color 0 0 0 0))
+  )
+  (wire (pts (xy 648.97 289.56) (xy 648.97 294.64))
+    (stroke (width 0) (type solid) (color 0 0 0 0))
+  )
+  (wire (pts (xy 648.97 294.64) (xy 648.97 297.18))
+    (stroke (width 0) (type solid) (color 0 0 0 0))
+  )
+  (wire (pts (xy 648.97 297.18) (xy 648.97 302.26))
+    (stroke (width 0) (type solid) (color 0 0 0 0))
+  )
+  (wire (pts (xy 648.97 302.26) (xy 648.97 304.8))
+    (stroke (width 0) (type solid) (color 0 0 0 0))
+  )
+  (wire (pts (xy 648.97 304.8) (xy 648.97 309.88))
+    (stroke (width 0) (type solid) (color 0 0 0 0))
+  )
+  (wire (pts (xy 648.97 309.88) (xy 648.97 312.42))
+    (stroke (width 0) (type solid) (color 0 0 0 0))
+  )
+  (wire (pts (xy 648.97 312.42) (xy 648.97 317.5))
+    (stroke (width 0) (type solid) (color 0 0 0 0))
+  )
+  (wire (pts (xy 648.97 317.5) (xy 648.97 320.04))
+    (stroke (width 0) (type solid) (color 0 0 0 0))
+  )
+  (wire (pts (xy 648.97 320.04) (xy 648.97 325.12))
+    (stroke (width 0) (type solid) (color 0 0 0 0))
+  )
+  (wire (pts (xy 648.97 325.12) (xy 648.97 327.66))
+    (stroke (width 0) (type solid) (color 0 0 0 0))
+  )
+  (wire (pts (xy 648.97 327.66) (xy 648.97 332.74))
+    (stroke (width 0) (type solid) (color 0 0 0 0))
+  )
+  (wire (pts (xy 648.97 332.74) (xy 648.97 335.28))
+    (stroke (width 0) (type solid) (color 0 0 0 0))
+  )
+  (wire (pts (xy 648.97 335.28) (xy 648.97 340.36))
+    (stroke (width 0) (type solid) (color 0 0 0 0))
+  )
+  (wire (pts (xy 648.97 340.36) (xy 648.97 342.9))
+    (stroke (width 0) (type solid) (color 0 0 0 0))
+  )
+  (wire (pts (xy 648.97 342.9) (xy 648.97 347.98))
+    (stroke (width 0) (type solid) (color 0 0 0 0))
+  )
+  (wire (pts (xy 648.97 347.98) (xy 648.97 350.52))
+    (stroke (width 0) (type solid) (color 0 0 0 0))
+  )
   (wire (pts (xy 722.63 76.2) (xy 744.22 76.2))
     (stroke (width 0) (type solid) (color 0 0 0 0))
@@
     )
   )
-  (symbol (lib_name "ECP5UM25:ECP5UM25_8") (lib_id "ECP5UM25:ECP5UM25") (at 455.295 71.12 0) (unit 1)
-    (in_bom yes) (on_board yes)
-    (property "Reference" "U1" (id 0) (at 500.9306 134.5503 0)
-      (effects (font (size 1.27 1.27)) (justify left))
-    )
-    (property "Value" "ECP5UM25" (id 1) (at 500.9306 136.849 0)
-      (effects (font (size 1.27 1.27)) (justify left))
-    )
-    (property "Footprint" "Package_BGA:Lattice_caBGA-381_17.0x17.0mm_Layout20x20_P0.8mm_Ball0.4mm_Pad0.4mm_NSMD" (id 2) (at 455.295 63.12 0)
-      (effects (font (size 1.27 1.27)) hide)
-    )
-    (property "Datasheet" "" (id 3) (at 455.295 71.12 0)
-      (effects (font (size 1.27 1.27)) hide)
-    )
+  (symbol (lib_name "ECP5UM25:ECP5UM25_8") (lib_id "ECP5UM25:ECP5UM25") (at 654.05 251.46 0) (unit 1)
+    (in_bom yes) (on_board yes)
+    (property "Reference" "U1" (id 0) (at 699.6856 314.8903 0)
+      (effects (font (size 1.27 1.27)) (justify left))
+    )
+    (property "Value" "ECP5UM25" (id 1) (at 699.6856 317.189 0)
+      (effects (font (size 1.27 1.27)) (justify left))
+    )
+    (property "Footprint" "Package_BGA:Lattice_caBGA-381_17.0x17.0mm_Layout20x20_P0.8mm_Ball0.4mm_Pad0.4mm_NSMD" (id 2) (at 654.05 243.46 0)
+      (effects (font (size 1.27 1.27)) hide)
+    )
+    (property "Datasheet" "" (id 3) (at 654.05 251.46 0)
+      (effects (font (size 1.27 1.27)) hide)
+    )

Commit message: changed RAM symbol, schematic of FT, USB PHY and VGA. Rerouted DRAM
Parts:
- added C21, C22, C23, C24, C25, C26, C27, C28, C29, C33, C34: 100n, Capacitor_SMD:C_0603_1608Metric, symbol Device:C_Small
- added C30, C31, C32: 4u7, Capacitor_SMD:C_0603_1608Metric, symbol Device:C_Small
- added C35, C36, C37, C38, C39: 470n, Capacitor_SMD:C_0402_1005Metric, symbol Device:C_Small
- added C40, C41, C42, C43, C44, C45, C46, C48, C49, C50, C51, C53, C54, C55: 100nF, Capacitor_SMD:C_0402_1005Metric, symbol Device:C_Small
- added C47, C52: 4u7, Capacitor_SMD:C_0402_1005Metric, symbol Device:C_Small
- added J1: USB_A, Connector_USB:USB_A_Molex_67643_Horizontal, symbol Connector:USB_A
- added J2: DB15_Female_HighDensity_MountingHoles, Connector_Dsub:DSUB-15-HD_Male_Horizontal_P2.29x1.98mm_EdgePinOffset3.03mm_Housed_MountingHolesOffset4.94mm, symbol Connector:DB15_Female_HighDensity_MountingHoles
- added L1, L2: L_Small, Inductor_SMD:L_0603_1608Metric, symbol Device:L_Small
- added R10: 12k +/-1%, Resistor_SMD:R_0603_1608Metric, symbol Device:R_Small
- added R100, R101, R102, R103, R104, R79, R80, R81, R82, R83, R84, R85, R86, R87, R88, R89, R90, R91, R92, R93, R94, R95, R96, R97, R98, R99: 51R, Resistor_SMD:R_0402_1005Metric, symbol Device:R_Small
- added R11, R12, R13, R14, R15, R16, R17, R18, R19, R20, R21, R22, R23, R24, R25, R26, R27, R28, R30, R31, R32, R33, R34, R35, R36, R37, R38, R39, R40, R41, R42, R43, R46, R47, R48, R49, R50, R51, R52, R53, R54, R55, R56, R57, R58, R59, R60, R61, R62, R63, R64, R65, R66, R67, R68, R69, R70, R71, R72, R73, R74, R75: R, Resistor_SMD:R_0402_1005Metric_Pad0.72x0.64mm_HandSolder, symbol Device:R_Small
- added R29: 1M, Resistor_SMD:R_0603_1608Metric, symbol Device:R_Small
- added R44, R45: 100R, Resistor_SMD:R_0402_1005Metric_Pad0.72x0.64mm_HandSolder, symbol Device:R_Small
- added R76, R77, R? (x2): 0R, Resistor_SMD:R_0402_1005Metric_Pad0.72x0.64mm_HandSolder, symbol Device:R_Small
- added R78: 12k 1%, Resistor_SMD:R_0603_1608Metric, symbol Device:R_Small
- added R9, R?: 10k, Resistor_SMD:R_0603_1608Metric, symbol Device:R_Small
- added R? (x4): 0R, Resistor_SMD:R_0603_1608Metric, symbol Device:R_Small
- added TP1: FTDI1V8REG, TestPoint:TestPoint_Pad_D1.5mm, symbol Connector:TestPoint
- added U4: FT2232HQ, Package_DFN_QFN:QFN-64-1EP_9x9mm_P0.5mm_EP4.35x4.35mm, symbol Interface_USB:FT2232HQ
- added U5: W25Q128JVS, Package_SO:SOIC-8_5.23x5.23mm_P1.27mm, symbol Memory_Flash:W25Q128JVS
- added U6, U7: USB3300-EZK, Package_DFN_QFN:QFN-32-1EP_5x5mm_P0.5mm_EP3.45x3.45mm, symbol Interface_USB:USB3300-EZK
- C1: value 0.1uF -> 4.7uF
- C10, C12, C14, C15, C17, C18, C19, C2, C20, C3, C4, C5, C7, C9: value 0.1uF -> 470n
- C11: value 0.1uF -> 100nF
- C16, C6, C8: value 4.7uF -> 470n
- R1: value 51R -> 0R; footprint Resistor_SMD:R_0402_1005Metric -> Resistor_SMD:R_0603_1608Metric
- R2: value 51R -> 240R
- R3: value 240R -> R; footprint Resistor_SMD:R_0402_1005Metric -> Resistor_SMD:R_0402_1005Metric_Pad0.72x0.64mm_HandSolder
- R4: value 0R -> R; footprint Resistor_SMD:R_1206_3216Metric_Pad1.30x1.75mm_HandSolder -> Resistor_SMD:R_0402_1005Metric_Pad0.72x0.64mm_HandSolder
- R6: footprint Resistor_SMD:R_1206_3216Metric_Pad1.30x1.75mm_HandSolder -> Resistor_SMD:R_0603_1608Metric
- R7, R8: value 51R -> R; footprint Resistor_SMD:R_0402_1005Metric -> Resistor_SMD:R_0402_1005Metric_Pad0.72x0.64mm_HandSolder
Connections:
- net DRAM_ADDR_0: now also R81.1
- net DRAM_ADDR_1: now also R82.1
- net DRAM_ADDR_10: now also R91.1
- net DRAM_ADDR_11: now also R92.1
- net DRAM_ADDR_12: now also R93.1
- net DRAM_ADDR_13: now also R94.1
- net DRAM_ADDR_14: now also R95.1
- net DRAM_ADDR_15: now also R96.1
- net DRAM_ADDR_2: now also R83.1
- net DRAM_ADDR_3: now also R84.1
- net DRAM_ADDR_4: now also R85.1
- net DRAM_ADDR_5: now also R86.1
- net DRAM_ADDR_6: now also R87.1
- net DRAM_ADDR_7: now also R88.1
- net DRAM_ADDR_8: now also R89.1
- net DRAM_ADDR_9: now also R90.1
- net DRAM_ADDR_BA0: now also R97.1
- net DRAM_ADDR_BA1: now also R98.1
- net DRAM_ADDR_BA2: now also R99.1
- net GND: now also R2.2, C21.2, C22.2, C23.2, C24.2, C25.2, C26.2, C27.2, C28.2, C29.2, C30.2, C31.2, C32.2, C33.2, C34.2, C35.2, C36.2, C37.2, C38.2, C39.2, C40.2, C41.2, C42.2, C43.2, C44.2, C45.2, C46.2, C47.2, C48.2, C49.2, C50.2, C51.2, C52.2, C53.2, C54.1, C55.2, J1.4 (GND), J1.5 (Shield), J2.10, J2.5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; no longer R3.2
- net at U2.L8 (ZQ): now also R2.1; no longer R3.1
- net BANK_AH_RDQS: no longer names the net of U1.E4 (PL8A/LDQS8/-)
- net BANK_AH_RDQS: no longer U3.C7 (UDQS)
- net BANK_AH_RDQSN: no longer names the net of U1.D5 (PL8B/LDQSN8/-)
- net BANK_AH_RDQSN: no longer U3.B7 (UDQS#)
- net BANK_AL_RDQS: no longer names the net of U1.H4 (PL20A/LDQS20/GR_PCLK7_1)
- net BANK_AL_RDQS: no longer U3.F3 (LDQS)
- net BANK_AL_RDQSN: no longer names the net of U1.G5 (PL20B/LDQSN20/-)
- net BANK_AL_RDQSN: no longer U3.G3 (LDQS#)
- net BANK_A_DQ0: no longer names the net of U1.A2 (PL14A/LDQ20/-)
- net BANK_A_DQ0: no longer U3.E3 (DQ0)
- net BANK_A_DQ1: no longer names the net of U1.B1 (PL14B/LDQ20/-)
- net BANK_A_DQ1: no longer U3.F7 (DQ1)
- net BANK_A_DQ10: no longer names the net of U1.A3 (PL5C/LDQ8/-)
- net BANK_A_DQ10: no longer U3.C8 (DQ10)
- net BANK_A_DQ11: no longer names the net of U1.B3 (PL5D/LDQ8/-)
- net BANK_A_DQ11: no longer U3.C2 (DQ11)
- net BANK_A_DQ12: no longer names the net of U1.F4 (PL11A/LDQ8/-)
- net BANK_A_DQ12: no longer U3.A7 (DQ12)
- net BANK_A_DQ13: no longer names the net of U1.E3 (PL11B/LDQ8/-)
- net BANK_A_DQ13: no longer U3.A2 (DQ13)
- net BANK_A_DQ14: no longer names the net of U1.E5 (PL11C/LDQ8/-)
- net BANK_A_DQ14: no longer U3.B8 (DQ14)
- net BANK_A_DQ15: no longer names the net of U1.F5 (PL11D/LDQ8/-)
- net BANK_A_DQ15: no longer U3.A3 (DQ15)
- net BANK_A_DQ2: no longer names the net of U1.C1 (PL17A/LDQ20/-)
- net BANK_A_DQ2: no longer U3.F2 (DQ2)
- net BANK_A_DQ3: no longer names the net of U1.D1 (PL17B/LDQ20/-)
- net BANK_A_DQ3: no longer U3.F8 (DQ3)
- net BANK_A_DQ4: no longer names the net of U1.G3 (PL23A/LDQ20/PCLKT7_1)
- net BANK_A_DQ4: no longer U3.H3 (DQ4)
- net BANK_A_DQ5: no longer names the net of U1.F3 (PL23B/LDQ20/PCLKC7_1)
- net BANK_A_DQ5: no longer U3.H8 (DQ5)
- net BANK_A_DQ6: no longer names the net of U1.F2 (PL23C/LDQ20/PCLKT7_0)
- net BANK_A_DQ6: no longer U3.G2 (DQ6)
- net BANK_A_DQ7: no longer names the net of U1.E2 (PL23D/LDQ20/PCLKC7_0)
- net BANK_A_DQ7: no longer U3.H7 (DQ7)
- net BANK_A_DQ8: no longer names the net of U1.C4 (PL5A/LDQ8/-)
- net BANK_A_DQ8: no longer U3.D7 (DQ8)
- net BANK_A_DQ9: no longer names the net of U1.B4 (PL5B/LDQ8/-)
- net BANK_A_DQ9: no longer U3.C3 (DQ9)
- net BANK_A_VREF: no longer names the net of U1.B2 (PL14C/LDQ20/VREF1_7)
- net BANK_BH_RDQS: no longer names the net of U1.F17 (PR8A/RDQS8/-)
- net BANK_BH_RDQS: no longer U2.C7 (UDQS)
- net BANK_BH_RDQSN: no longer names the net of U1.G18 (PR8B/RDQSN8/-)
- net BANK_BH_RDQSN: no longer U2.B7 (UDQS#)
- net BANK_BL_RDQS: no longer names the net of U1.G19 (PR20A/RDQS20/GR_PCLK2_1)
- net BANK_BL_RDQS: no longer U2.F3 (LDQS)
- net BANK_BL_RDQSN: no longer names the net of U1.H20 (PR20B/RDQSN20/-)
- net BANK_BL_RDQSN: no longer U2.G3 (LDQS#)
- net BANK_B_DQ0: no longer names the net of U1.C20 (PR14A/RDQ20/-)
- net BANK_B_DQ0: no longer U2.E3 (DQ0)
- net BANK_B_DQ1: no longer names the net of U1.D19 (PR14B/RDQ20/-)
- net BANK_B_DQ1: no longer U2.F7 (DQ1)
- net BANK_B_DQ10: no longer names the net of U1.E18 (PR5C/RDQ8/-)
- net BANK_B_DQ10: no longer U2.C8 (DQ10)
- net BANK_B_DQ11: no longer names the net of U1.F18 (PR5D/RDQ8/-)
- net BANK_B_DQ11: no longer U2.C2 (DQ11)
- net BANK_B_DQ12: no longer names the net of U1.H18 (PR11A/RDQ8/-)
- net BANK_B_DQ12: no longer U2.A7 (DQ12)
- net BANK_B_DQ13: no longer names the net of U1.H17 (PR11B/RDQ8/-)
- net BANK_B_DQ13: no longer U2.A2 (DQ13)
- net BANK_B_DQ14: no longer names the net of U1.J17 (PR11C/RDQ8/-)
- net BANK_B_DQ14: no longer U2.B8 (DQ14)
- net BANK_B_DQ15: no longer names the net of U1.J16 (PR11D/RDQ8/-)
- net BANK_B_DQ15: no longer U2.A3 (DQ15)
- net BANK_B_DQ2: no longer names the net of U1.E20 (PR17A/RDQ20/-)
- net BANK_B_DQ2: no longer U2.F2 (DQ2)
- net BANK_B_DQ3: no longer names the net of U1.F19 (PR17B/RDQ20/-)
- net BANK_B_DQ3: no longer U2.F8 (DQ3)
- net BANK_B_DQ4: no longer names the net of U1.J19 (PR23A/RDQ20/PCLKT2_1)
- net BANK_B_DQ4: no longer U2.H3 (DQ4)
- net BANK_B_DQ5: no longer names the net of U1.K19 (PR23B/RDQ20/PCLKC2_1)
- net BANK_B_DQ5: no longer U2.H8 (DQ5)
- net BANK_B_DQ6: no longer names the net of U1.J20 (PR23C/RDQ20/PCLKT2_0)
- net BANK_B_DQ6: no longer U2.G2 (DQ6)
- net BANK_B_DQ7: no longer names the net of U1.K20 (PR23D/RDQ20/PCLKC2_0)
- net BANK_B_DQ7: no longer U2.H7 (DQ7)
- net BANK_B_DQ8: no longer names the net of U1.D18 (PR5A/RDQ8/-)
- net BANK_B_DQ8: no longer U2.D7 (DQ8)
- net BANK_B_DQ9: no longer names the net of U1.E17 (PR5B/RDQ8/-)
- net BANK_B_DQ9: no longer U2.C3 (DQ9)
- net BANK_B_VREF: no longer names the net of U1.D20 (PR14C/RDQ20/VREF1_2)
- net DRAMREF renamed DRAM_VREF
- net DRAM_VREF: now also C40.1, C41.1, C42.1; no longer C1.1, C14.1, C17.1, C2.1, C3.1
- net DRAM_A_CKE: no longer names the net of U1.C3 (PL8C/LDQ8/-)
- net DRAM_A_CKE: no longer U3.K9 (CKE)
- removed net DRAM_A_CK_N: R8.1, U1.A4 (PL2A/LDQ8/-), U3.K7 (CK#)
- removed net DRAM_A_CK_P: R7.1, U1.A5 (PL2B/LDQ8/-), U3.J7 (CK)
- net DRAM_A_LDM: no longer names the net of U1.H3 (PL20D/LDQ20/-)
- net DRAM_A_LDM: no longer U3.E7 (LDM)
- net DRAM_A_ODT: no longer names the net of U1.D3 (PL8D/LDQ8/-)
- net DRAM_A_ODT: no longer U3.K1 (ODT)
- net DRAM_A_UDM: no longer names the net of U1.H5 (PL20C/LDQ20/GR_PCLK7_0)
- net DRAM_A_UDM: no longer U3.D3 (UDM)
- net DRAM_A_nCAS: no longer names the net of U1.B5 (PL2C/LDQ8/-)
- net DRAM_A_nCAS: no longer U3.K3 (CAS#)
- net DRAM_A_nCS: no longer names the net of U1.D2 (PL17C/LDQ20/-)
- net DRAM_A_nCS: no longer U3.L2 (CS#)
- net DRAM_A_nRAS: no longer names the net of U1.C5 (PL2D/LDQ8/-)
- net DRAM_A_nRAS: no longer U3.J3 (RAS#)
- net DRAM_A_nRESET: no longer names the net of U1.C2 (PL14D/LDQ20/-)
- net DRAM_A_nRESET: no longer U3.T2 (RESET#)
- net DRAM_A_nWE: no longer names the net of U1.E1 (PL17D/LDQ20/-)
- net DRAM_A_nWE: no longer U3.L3 (WE#)
- net DRAM_B_CKE: no longer names the net of U1.G16 (PR8C/RDQ8/-)
- net DRAM_B_CKE: no longer U2.K9 (CKE)
- removed net DRAM_B_CK_N: R2.1, U1.C18 (PR2A/RDQ8/-), U2.K7 (CK#)
- removed net DRAM_B_CK_P: R1.1, U1.D17 (PR2B/RDQ8/S0_IN), U2.J7 (CK)
- net DRAM_B_LDM: no longer names the net of U1.K18 (PR20D/RDQ20/-)
- net DRAM_B_LDM: no longer U2.E7 (LDM)
- net DRAM_B_ODT: no longer names the net of U1.H16 (PR8D/RDQ8/-)
- net DRAM_B_ODT: no longer U2.K1 (ODT)
- net DRAM_B_UDM: no longer names the net of U1.J18 (PR20C/RDQ20/GR_PCLK2_0)
- net DRAM_B_UDM: no longer U2.D3 (UDM)
- net DRAM_B_nCAS: no longer names the net of U1.E16 (PR2C/RDQ8/-)
- net DRAM_B_nCAS: no longer U2.K3 (CAS#)
- net DRAM_B_nCS: no longer names the net of U1.F20 (PR17C/RDQ20/-)
- net DRAM_B_nCS: no longer U2.L2 (CS#)
- net DRAM_B_nRAS: no longer names the net of U1.F16 (PR2D/RDQ8/-)
- net DRAM_B_nRAS: no longer U2.J3 (RAS#)
- net DRAM_B_nRESET: no longer names the net of U1.E19 (PR14D/RDQ20/-)
- net DRAM_B_nRESET: no longer U2.T2 (RESET#)
- net DRAM_B_nWE: no longer names the net of U1.G20 (PR17D/RDQ20/-)
- net DRAM_B_nWE: no longer U2.L3 (WE#)
- net DRAM_SUPPLY_A: no longer names the net of C13.1, C16.1, C19.1, U3.A1 (Vddq), U3.A8 (Vddq), U3.B2 (Vdd), U3.C1 (Vddq), U3.C9 (Vddq), U3.D2 (Vddq), U3.D9 (Vdd), U3.E9 (Vddq), U3.F1 (Vddq), U3.G7 (Vdd), U3.H2 (Vddq), U3.H9 (Vddq), U3.K2 (Vdd), U3.K8 (Vdd), U3.N1 (Vdd), U3.N9 (Vdd), U3.R1 (Vdd), U3.R9 (Vdd)
- net DRAM_SUPPLY_A: now also C10.1, C14.1, C17.1, C4.1, C6.1, C8.1, R6.1, C35.1, C37.1, C39.1; no longer C12.1, C15.1, C18.1, R6.2
- net DRAM_SUPPLY_B: no longer names the net of C5.1, C7.1, C9.1, U2.A1 (Vddq), U2.A8 (Vddq), U2.B2 (Vdd), U2.C1 (Vddq), U2.C9 (Vddq), U2.D2 (Vddq), U2.D9 (Vdd), U2.E9 (Vddq), U2.F1 (Vddq), U2.G7 (Vdd), U2.H2 (Vddq), U2.H9 (Vddq), U2.K2 (Vdd), U2.K8 (Vdd), U2.N1 (Vdd), U2.N9 (Vdd), U2.R1 (Vdd), U2.R9 (Vdd)
- net DRAM_SUPPLY_B: now also C1.1, C12.1, C15.1, C18.1, C2.1, C20.1, C3.1, R1.1, C36.1, C38.1; no longer C10.1, C6.1, C8.1, R4.2
- removed net DRAM_SUPPLY_GLOB: R4.1, R6.1, U1.H14 (VCCIO2/-), U1.H15 (VCCIO2/-), U1.J15 (VCCIO2/-)
- new net: R10.2, U4.6 (REF)
- new net: R36.2, R43.1
- new net: R?.1, U4.19 (ADBUS3)
- new net: R33.2, R40.1
- new net: R40.2, R48.2, R49.1
- new net: R41.2, R49.2, R50.1
- new net: R62.2, R68.2, R69.1
- new net: R?.1, U4.16 (ADBUS0)
- new net: R?.1, U4.17 (ADBUS1)
- new net: R9.2, U4.14 (~RESET)
- new net: C55.1, R79.2, R80.2
- new net: R63.2, R69.2, R70.1
- new net: R64.2, R70.2, R71.1
- new net: R42.2, R50.2, R51.1
- new net: R30.2, R37.1
- new net: R57.2, R64.1
- new net: J2.14, R45.1
- new net: R59.2, R66.1
- new net: C31.1, C32.1, L2.2, U4.4 (VPHY)
- new net: R11.2, R18.1
- new net: R39.2, R47.2, R48.1
- new net: R60.2, R67.1
- new net: R67.2, R73.2, R74.2
- new net: R16.2, R22.2, R23.1
- new net: R17.2, R23.2, R24.1
- new net: C33.1, C34.1, L1.2, U4.9 (VPLL)
- new net: R34.2, R41.1
- new net: C53.1, U7.15 (VDD1.8), U7.26 (VDD1.8)
- new net: C54.2, U7.29 (VDDA1.8)
- new net: R78.2, U7.32 (RBIAS)
- new net: R76.1, R77.1, U7.5 (ID)
- new net: R74.1, R75.2
- new net: R31.2, R38.1
- new net: R38.2, R46.2, R47.1
- new net: R55.2, R62.1
- new net: R15.2, R21.2, R22.1
- new net: R14.1, R3.2
- new net: R32.2, R39.1
- new net: R?.1, R?.1, U6.5 (ID)
- new net: R43.2, R51.2, R52.2
- new net: C29.1, C30.1, TP1.1, U4.49 (VREGOUT)
- new net: R65.2, R71.2, R72.1
- new net: R66.2, R72.2, R73.1
- new net: R13.2, R20.1
- new net: R20.2, R26.2, R27.2
- new net: R18.2, R24.2, R25.1
- new net: R35.2, R42.1
- new net: R12.2, R19.1
- new net: R58.2, R65.1
- new net: R17.1, R8.2
- new net: R16.1, R7.2
- new net: R15.1, R4.2
- new net: R?.1, U4.18 (ADBUS2)
- new net: R54.2, R61.1
- new net: R27.1, R28.2
- new net: R56.2, R63.1
- new net: J2.13, R44.1
- new net: R19.2, R25.2, R26.1
- new net: R52.1, R53.2
- new net: J2.0, R29.2
- new net +1V35: R1.2, R6.2
- new net +1V8: C22.1, C23.1, C24.1, U4.12 (VCORE), U4.37 (VCORE), U4.64 (VCORE)
- new net +3V3: C21.1, C25.1, C26.1, C27.1, C28.1, C43.1, C44.1, C45.1, C46.1, C47.1, C48.1, C49.1, C50.1, C51.1, C52.1, L1.1, L2.1, R76.2, R9.1, R?.2, U4.20 (VCCIO), U4.31 (VCCIO), U4.42 (VCCIO), U4.50 (VREGIN), U4.56 (VCCIO), U6.16 (VDD3.3), U6.25 (VDD3.3), U6.30 (VDD3.3), U6.6 (VDD3.3), U7.16 (VDD3.3), U7.25 (VDD3.3), U7.30 (VDD3.3), U7.31 (REG_EN), U7.6 (VDD3.3)
- new net DRAM_CKE: U2.K9 (CKE), U3.K9 (CKE)
- new net DRAM_CLK_N: R79.1, U2.K7 (CK#), U3.K7 (CK#)
- new net DRAM_CLK_P: R80.1, U2.J7 (CK), U3.J7 (CK)
- new net DRAM_DATA_0: U2.E3 (DQ0)
- new net DRAM_DATA_1: U2.F7 (DQ1)
- new net DRAM_DATA_10: U2.C8 (DQ10)
- new net DRAM_DATA_11: U2.C2 (DQ11)
- new net DRAM_DATA_12: U2.A7 (DQ12)
- new net DRAM_DATA_13: U2.A2 (DQ13)
- new net DRAM_DATA_14: U2.B8 (DQ14)
- new net DRAM_DATA_15: U2.A3 (DQ15)
- new net DRAM_DATA_16: U3.E3 (DQ0)
- new net DRAM_DATA_17: U3.F7 (DQ1)
- new net DRAM_DATA_18: U3.F2 (DQ2)
- new net DRAM_DATA_19: U3.F8 (DQ3)
- new net DRAM_DATA_2: U2.F2 (DQ2)
- new net DRAM_DATA_20: U3.H3 (DQ4)
- new net DRAM_DATA_21: U3.H8 (DQ5)
- new net DRAM_DATA_22: U3.G2 (DQ6)
- new net DRAM_DATA_23: U3.H7 (DQ7)
- new net DRAM_DATA_24: U3.D7 (DQ8)
- new net DRAM_DATA_25: U3.C3 (DQ9)
- new net DRAM_DATA_26: U3.C8 (DQ10)
- new net DRAM_DATA_27: U3.C2 (DQ11)
- new net DRAM_DATA_28: U3.A7 (DQ12)
- new net DRAM_DATA_29: U3.A2 (DQ13)
- new net DRAM_DATA_3: U2.F8 (DQ3)
- new net DRAM_DATA_30: U3.B8 (DQ14)
- new net DRAM_DATA_31: U3.A3 (DQ15)
- new net DRAM_DATA_4: U2.H3 (DQ4)
- new net DRAM_DATA_5: U2.H8 (DQ5)
- new net DRAM_DATA_6: U2.G2 (DQ6)
- new net DRAM_DATA_7: U2.H7 (DQ7)
- new net DRAM_DATA_8: U2.D7 (DQ8)
- new net DRAM_DATA_9: U2.C3 (DQ9)
- new net DRAM_DM0: U2.E7 (LDM)
- new net DRAM_DM1: U2.D3 (UDM)
- new net DRAM_DM2: U3.E7 (LDM)
- new net DRAM_DM3: U3.D3 (UDM)
- new net DRAM_DQS0_N: U2.G3 (LDQS#)
- new net DRAM_DQS0_P: U2.F3 (LDQS)
- new net DRAM_DQS1_N: U2.B7 (UDQS#)
- new net DRAM_DQS1_P: U2.C7 (UDQS)
- new net DRAM_DQS2_N: U3.G3 (LDQS#)
- new net DRAM_DQS2_P: U3.F3 (LDQS)
- new net DRAM_DQS3_N: U3.B7 (UDQS#)
- new net DRAM_DQS3_P: U3.C7 (UDQS)
- new net DRAM_ODT: R101.1, U2.K1 (ODT), U3.K1 (ODT)
- new net DRAM_nCAS: R103.1, U2.K3 (CAS#), U3.K3 (CAS#)
- new net DRAM_nCS: R100.1, U2.L2 (CS#), U3.L2 (CS#)
- new net DRAM_nRAS: R102.1, U2.J3 (RAS#), U3.J3 (RAS#)
- new net DRAM_nRESET: U2.T2 (RESET#), U3.T2 (RESET#)
- new net DRAM_nWE: R104.1, U2.L3 (WE#), U3.L3 (WE#)
- new net FIFO_D0/RX: U4.38 (BDBUS0)
- new net FIFO_D1/TX: U4.39 (BDBUS1)
- new net FIFO_D2: U4.40 (BDBUS2)
- new net FIFO_D3: U4.41 (BDBUS3)
- new net FIFO_D4: U4.43 (BDBUS4)
- new net FIFO_D5: U4.44 (BDBUS5)
- new net FIFO_D6: U4.45 (BDBUS6)
- new net FIFO_D7: U4.46 (BDBUS7)
- new net FIFO_WKUP: U4.55 (BCBUS4)
- new net FIFO_nRD: U4.53 (BCBUS2)
- new net FIFO_nRXE: U4.48 (BCBUS0)
- new net FIFO_nTXE: U4.52 (BCBUS1)
- new net FIFO_nWR: U4.54 (BCBUS3)
- new net JTAG_TCK: R?.2, R?.2
- new net JTAG_TDI: R?.2
- new net JTAG_TDO: R?.2
- new net JTAG_TMS: R?.2
- new net USB_FPGA_N: U6.8 (DM)
- new net USB_FPGA_P: U6.7 (DP)
- new net USB_FTDI_N: U4.7 (DM)
- new net USB_FTDI_P: U4.8 (DP)
- new net USB_HOST_CLK: U7.28 (XI)
- new net USB_HOST_CLKOUT: U7.14 (CLKOUT)
- new net USB_HOST_DATA0: U7.24 (DATA0)
- new net USB_HOST_DATA1: U7.23 (DATA1)
- new net USB_HOST_DATA2: U7.22 (DATA2)
- new net USB_HOST_DATA3: U7.21 (DATA3)
- new net USB_HOST_DATA4: U7.20 (DATA4)
- new net USB_HOST_DATA5: U7.19 (DATA5)
- new net USB_HOST_DATA6: U7.18 (DATA6)
- new net USB_HOST_DATA7: U7.17 (DATA7)
- new net USB_HOST_DIR: U7.12 (DIR)
- new net USB_HOST_N: J1.2 (D-), U7.8 (DM)
- new net USB_HOST_NXT: U7.11 (NXT)
- new net USB_HOST_P: J1.3 (D+), U7.7 (DP)
- new net USB_HOST_RESET: U7.9 (RESET)
- new net USB_HOST_STP: U7.13 (STP)
- new net USB_SLAVE_CLK: U6.28 (XI)
- new net USB_SLAVE_CLKOUT: U6.14 (CLKOUT)
- new net USB_SLAVE_DATA0: U6.24 (DATA0)
- new net USB_SLAVE_DATA1: U6.23 (DATA1)
- new net USB_SLAVE_DATA2: U6.22 (DATA2)
- new net USB_SLAVE_DATA3: U6.21 (DATA3)
- new net USB_SLAVE_DATA4: U6.20 (DATA4)
- new net USB_SLAVE_DATA5: U6.19 (DATA5)
- new net USB_SLAVE_DATA6: U6.18 (DATA6)
- new net USB_SLAVE_DATA7: U6.17 (DATA7)
- new net USB_SLAVE_DIR: U6.12 (DIR)
- new net USB_SLAVE_NXT: U6.11 (NXT)
- new net USB_SLAVE_RESET: U6.9 (RESET)
- new net USB_SLAVE_STP: U6.13 (STP)
- new net VGA_AB: J2.3, R61.2, R68.1
- new net VGA_AG: J2.2, R37.2, R46.1
- new net VGA_AR: J2.1, R14.2, R21.1
- new net VGA_BUF_B_0: R54.1
- new net VGA_BUF_B_1: R55.1
- new net VGA_BUF_B_2: R56.1
- new net VGA_BUF_B_3: R57.1
- new net VGA_BUF_B_4: R58.1
- new net VGA_BUF_B_5: R59.1
- new net VGA_BUF_B_6: R60.1
- new net VGA_BUF_G_0: R30.1
- new net VGA_BUF_G_1: R31.1
- new net VGA_BUF_G_2: R32.1
- new net VGA_BUF_G_3: R33.1
- new net VGA_BUF_G_4: R34.1
- new net VGA_BUF_G_5: R35.1
- new net VGA_BUF_G_6: R36.1
- new net VGA_BUF_R_0: R3.1
- new net VGA_BUF_R_1: R4.1
- new net VGA_BUF_R_2: R7.1
- new net VGA_BUF_R_3: R8.1
- new net VGA_BUF_R_4: R11.1
- new net VGA_BUF_R_5: R12.1
- new net VGA_BUF_R_6: R13.1
- new net VGA_HSYNC: R44.2
- new net VGA_VSYNC: R45.2
- no-connect marks 26 -> 52
Other:
- note added: "ADBUS4-5 and ACBUS as GPIO. Should we connect some leds here? ALSO, this can be used as reset"
- note added: "DRAM"
- note added: "For termination refer to https://www.ti.com/lit/an/sprabi1c/sprabi1c.pdf page 16"
- note added: "For topology refer to https://www.ti.com/lit/an/sprabi1c/sprabi1c.pdf page 14"
- note added: "IFACE voltage 3V3"
- note added: "POPULATE PREFIX depending on resolution"
- note added: "Route address and control as fly-by. Terminate at end"
- note added: "TODO: flash"
- note added: "TODO: oscylator"
- note added: "USB HOST UART/JTAG"
- note added: "USB HOSTPHY"
- note added: "USB PER PHY"
- note added: "always populate"
- note added: "consult https://digilent.com/reference/_media/reference/pmod/pmodvga/pmodvga_sch.pdf"
- note added: "place close to power pins"
- note added: "populate unused with 0R"
- note added: "refer to https://ftdichip.com/wp-content/uploads/2020/07/DS_FT2232H.pdf page 14, pins configured as MPSSE -> JTAG."
- note added: "refer to https://ftdichip.com/wp-content/uploads/2020/07/DS_FT2232H.pdf page 15, pins configured as a CPU-stype FIFO interface."
- note added: "refer to https://pl.mouser.com/datasheet/2/268/MCHP_S_A0002336793_1-2521138.pdf page 41"
- note added: "refer to page 9 for XI 24MHz"
- note added: "use any reasonable value (all same)"
- note removed: "DRAM A SUPPLY"
- note removed: "DRAM B SUPPLY"
- moved on the sheet: C11, C13, C16, R5, R6, U1C, U1D, U1E, U1F, U1G, U1H, U1I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

Commit message: VGA phy schematic and layout
Parts:
- removed R13, R20, R26, R36, R43, R51, R60, R67, R73: R, Resistor_SMD:R_0402_1005Metric_Pad0.72x0.64mm_HandSolder, symbol Device:R_Small
- added U10, U8, U9: SN74ALVC245PWR, Package_SO:TSSOP-20_4.4x6.5mm_P0.65mm, symbol SN74ALVC245PWR:SN74ALVC245PWR
- gave numbers to parts that had none: 7
Connections:
- net GND: now also U10.10 (GND), U8.10 (GND), U9.10 (GND)
- net VGA_BUF_B_0: now also U8.12 (B7)
- net VGA_BUF_B_1: now also U8.11 (B8)
- net VGA_BUF_B_2: now also U9.14 (B5)
- net VGA_BUF_B_3: now also U9.13 (B6)
- net VGA_BUF_B_4: now also U10.14 (B5)
- net VGA_BUF_B_5: now also U10.13 (B6)
- net VGA_BUF_G_0: now also U8.14 (B5)
- net VGA_BUF_G_1: now also U8.13 (B6)
- net VGA_BUF_G_2: now also U9.16 (B3)
- net VGA_BUF_G_3: now also U9.15 (B4)
- net VGA_BUF_G_4: now also U10.16 (B3)
- net VGA_BUF_G_5: now also U10.15 (B4)
- net VGA_BUF_R_0: now also U8.16 (B3)
- net VGA_BUF_R_1: now also U8.15 (B4)
- net VGA_BUF_R_2: now also U9.18 (B1)
- net VGA_BUF_R_3: now also U9.17 (B2)
- net VGA_BUF_R_4: now also U10.18 (B1)
- net VGA_BUF_R_5: now also U10.17 (B2)
- net VGA_HSYNC: now also U8.18 (B1)
- net VGA_VSYNC: now also U8.17 (B2)
- net at R42.2, R50.2: now also R52.2
- net at R74.2: now also R66.2, R72.2
- net at R27.2: now also R19.2, R25.2
Other:
- moved on the sheet: J2, R11, R12, R14, R15, R16, R17, R18, R19, R21, R22, R23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

Commit message: power failure
Parts:
- removed R100, R101, R102, R103, R104, R81, R82, R83, R84, R85, R86, R87, R88, R89, R90, R91, R92, R93, R94, R95, R96, R97, R98, R99: 51R, Resistor_SMD:R_0402_1005Metric, symbol Device:R_Small
- added C56, C57, C59, C60: 100nF, Capacitor_SMD:C_0402_1005Metric, symbol Device:C_Small
- added C58: 470n, Capacitor_SMD:C_0402_1005Metric, symbol Device:C_Small
- added C61, C62: 4u7, Capacitor_SMD:C_0603_1608Metric, symbol Device:C_Small
- added C63, C64, C65: 4u7, Capacitor_SMD:C_0402_1005Metric, symbol Device:C_Small
- added J10, J11, J12, J8, J9: AudioJack3_Ground_Switch, Connector_Audio:Jack_3.5mm_CUI_SJ1-3535NG_Horizontal, symbol Connector:AudioJack3_Ground_Switch
- added J3: Bus_PCI_Express_x1, Connector_PCBEdge:BUS_PCIexpress_x1, symbol Connector:Bus_PCI_Express_x1
- added J4: 1367073-1, Connector:Connector_SFP_and_Cage, symbol 1367073-1:1367073-1
- added J5: RJ45_LED_Shielded, Connector_RJ:RJ45_Amphenol_RJHSE538X, symbol Connector:RJ45_LED_Shielded
- added J6: USB_C_Receptacle, Connector_USB:USB_C_Receptacle_GCT_USB4085, symbol Connector:USB_C_Receptacle
- added J7: MEM2051-00-195-00-A, footprints:MEM2051-00-195-00-A, symbol MEM2051-00-195-00-A:MEM2051-00-195-00-A
- added R13: 12k 1%, Resistor_SMD:R_0603_1608Metric, symbol Device:R_Small
- added R20: 10k, Resistor_SMD:R_0402_1005Metric_Pad0.72x0.64mm_HandSolder, symbol Device:R_Small
- added R26, R36: 1k, Resistor_SMD:R_0402_1005Metric_Pad0.72x0.64mm_HandSolder, symbol Device:R_Small
- added RN1, RN2, RN4, RN5, RN6, RN7: 51R, symbol Device:R_Pack04_Split
- added RN3, RN8: 51R, Resistor_SMD:R_Array_Concave_4x0402, symbol Device:R_Pack04_Split
- added TP2: 1V8, TestPoint:TestPoint_Pad_D1.0mm, symbol Connector:TestPoint
- added U11: KSZ9021RL, Package_QFP:LQFP-64-1EP_10x10mm_P0.5mm_EP6.5x6.5mm, symbol KSZ9021RL:KSZ9021RL
- added U12: TUSB2036, Package_QFP:LQFP-32_7x7mm_P0.8mm, symbol Interface_USB:TUSB2036
- added U13: TPS2041B, Package_TO_SOT_SMD:SOT-23-5, symbol Power_Management:TPS2041B
- J1: footprint Connector_USB:USB_A_Molex_67643_Horizontal -> Connector_USB:USB_A_Wuerth_614004134726_Horizontal
Connections:
- net +1V35: now also U1.H14 (VCCIO2/-), U1.H15 (VCCIO2/-), U1.J15 (VCCIO2/-), U1.L14 (VCCIO3/-), U1.L15 (VCCIO3/-), U1.M15 (VCCIO3/-)
- net +3V3: now also U10.20 (VCC), U5.8 (VCC), U6.31 (REG_EN), U8.20 (VCC), U9.20 (VCC), C58.1, C63.1, C64.1, C65.1
- net DRAM_ADDR_0: now also U1.E17 (PR5B/RDQ8/-), RN2.3 (R3.1)
- net DRAM_ADDR_1: now also U1.T18 (PR44D/RDQ44/-), RN7.3 (R3.1)
- net DRAM_ADDR_10: now also U1.U16 (PR47C/RDQ44/LRC_GPLL0T_IN), RN8.3 (R3.1)
- net DRAM_ADDR_11: now also U1.R17 (PR35D/RDQ32/-), RN6.1 (R1.1)
- net DRAM_ADDR_12: now also U1.U18 (PR47A/RDQ44/-), RN8.4 (R4.1)
- net DRAM_ADDR_13: now also U1.J16 (PR11D/RDQ8/-), RN1.1 (R1.1)
- net DRAM_ADDR_14: now also U1.L17 (PR29B/RDQ32/-), RN6.3 (R3.1)
- net DRAM_ADDR_15: now also U1.U17 (PR47B/RDQ44/-), RN7.1 (R1.1)
- net DRAM_ADDR_2: now also RN2.1 (R1.1)
- net DRAM_ADDR_3: now also U1.E16 (PR2C/RDQ8/-), RN2.2 (R2.1)
- net DRAM_ADDR_4: now also U1.R16 (PR35C/RDQ32/-), RN7.4 (R4.1)
- net DRAM_ADDR_5: now also RN1.4 (R4.1)
- net DRAM_ADDR_6: now also U1.L18 (PR29C/RDQ32/GR_PCLK3_1), RN6.2 (R2.1)
- net DRAM_ADDR_7: now also RN1.2 (R2.1)
- net DRAM_ADDR_8: now also U1.L16 (PR29A/RDQ32/GR_PCLK3_0), RN6.4 (R4.1)
- net DRAM_ADDR_9: now also U1.J17 (PR11C/RDQ8/-), RN1.3 (R3.1)
- net DRAM_ADDR_BA0: now also U1.D17 (PR2B/RDQ8/S0_IN), RN4.1 (R1.1)
- net DRAM_ADDR_BA1: now also U1.T17 (PR47D/RDQ44/LRC_GPLL0C_IN), RN7.2 (R2.1)
- net DRAM_ADDR_BA2: now also U1.D18 (PR5A/RDQ8/-), RN2.4 (R4.1)
- net DRAM_DQS0_N: now also U1.R18 (PR44B/RDQSN44/-)
- net DRAM_DQS0_P: now also U1.T19 (PR44A/RDQS44/-)
- net DRAM_DQS1_N: now also U1.M17 (PR32B/RDQSN32/-)
- net DRAM_DQS1_P: now also U1.N16 (PR32A/RDQS32/-)
- net DRAM_ODT: now also RN4.4 (R4.1)
- net DRAM_nCAS: now also RN5.1 (R1.1)
- net DRAM_nCS: now also U1.C20 (PR14A/RDQ20/-), RN4.2 (R2.1)
- net DRAM_nRAS: now also RN5.2 (R2.1)
- net DRAM_nWE: now also U1.C18 (PR2A/RDQ8/-), RN4.3 (R3.1)
- net FIFO_D0/RX: now also U1.B3 (PL5D/LDQ8/-)
- net FIFO_D1/TX: now also U1.A2 (PL14A/LDQ20/-)
- net FIFO_D2: now also U1.B4 (PL5B/LDQ8/-)
- net FIFO_D3: now also U1.A3 (PL5C/LDQ8/-)
- net FIFO_D4: now also U1.B5 (PL2C/LDQ8/-)
- net FIFO_D5: now also U1.A4 (PL2A/LDQ8/-)
- net FIFO_D6: now also U1.C5 (PL2D/LDQ8/-)
- net FIFO_D7: now also U1.A5 (PL2B/LDQ8/-)
- net FIFO_WKUP: now also U1.E5 (PL11C/LDQ8/-)
- net FIFO_nRD: now also U1.D5 (PL8B/LDQSN8/-)
- net FIFO_nRXE: now also U1.C4 (PL5A/LDQ8/-)
- net FIFO_nTXE: now also U1.C3 (PL8C/LDQ8/-)
- net FIFO_nWR: now also U1.D3 (PL8D/LDQ8/-)
- net GND: now also U5.4 (GND), C56.2, C57.1, C58.2, C59.2, C60.2, C61.2, C62.2, C63.2, C64.2, C65.2, R13.1, R20.2, RN1.5 (R4.2), RN1.6 (R3.2), RN1.7 (R2.2), RN1.8 (R1.2), RN2.5 (R4.2), RN2.6 (R3.2), RN2.7 (R2.2), RN2.8 (R1.2), RN4.5 (R4.2), RN4.6 (R3.2), RN4.7 (R2.2), RN4.8 (R1.2), RN5.7 (R2.2), RN5.8 (R1.2), RN6.5 (R4.2), RN6.6 (R3.2), RN6.7 (R2.2), RN6.8 (R1.2), RN7.5 (R4.2), RN7.6 (R3.2), RN7.7 (R2.2), RN7.8 (R1.2), RN8.5 (R4.2), RN8.6 (R3.2), U11.17 (VSS), U11.18 (VSS), U11.23 (VSS), U11.28 (VSS), U11.3 (AGNDH), U11.34 (VSS), U11.39 (VSS), U11.53 (VSS), U11.63 (AGNDH_BG), U11.65 (EP), U11.9 (AGNDH), U12.28 (GND), U12.7 (GND), U13.2 (GND)
- net USB_FPGA_N: now also U12.19 (DM3)
- net USB_FPGA_P: now also U12.20 (DP3)
- net USB_SLAVE_CLK: now also U1.E4 (PL8A/LDQS8/-)
- net USB_SLAVE_CLKOUT: now also U1.F5 (PL11D/LDQ8/-)
- net USB_SLAVE_DATA0: now also U1.B1 (PL14B/LDQ20/-)
- net USB_SLAVE_DATA1: now also U1.B2 (PL14C/LDQ20/VREF1_7)
- net USB_SLAVE_DATA2: now also U1.C1 (PL17A/LDQ20/-)
- net USB_SLAVE_DATA3: now also U1.C2 (PL14D/LDQ20/-)
- net USB_SLAVE_DATA4: now also U1.D1 (PL17B/LDQ20/-)
- net USB_SLAVE_DATA5: now also U1.D2 (PL17C/LDQ20/-)
- net USB_SLAVE_DATA6: now also U1.E1 (PL17D/LDQ20/-)
- net USB_SLAVE_DATA7: now also U1.E2 (PL23D/LDQ20/PCLKC7_0)
- net USB_SLAVE_DIR: now also U1.F4 (PL11A/LDQ8/-)
- net USB_SLAVE_NXT: now also U1.F3 (PL23B/LDQ20/PCLKC7_1)
- net USB_SLAVE_RESET: now also U1.E3 (PL11B/LDQ8/-)
- net USB_SLAVE_STP: now also U1.G3 (PL23A/LDQ20/PCLKT7_1)
- net VGA_HSYNC: now also U1.P4 (PL47D/LDQ44/LLC_GPLL0C_IN), U8.2 (A1); no longer R44.2, U8.18 (B1)
- net VGA_VSYNC: now also U1.P3 (PL47C/LDQ44/LLC_GPLL0T_IN), U8.3 (A2); no longer R45.2, U8.17 (B2)
- net DRAM_2_VCORE: now reaches C10.1, C13.1, C14.1, C16.1, C17.1, C19.1, C35.1, C37.1, C39.1, C4.1, C6.1, C8.1, R6.1, U3.A1 (Vddq), U3.A8 (Vddq), U3.B2 (Vdd), U3.C1 (Vddq), U3.C9 (Vddq), U3.D2 (Vddq), U3.D9 (Vdd), U3.E9 (Vddq), U3.F1 (Vddq), U3.G7 (Vdd), U3.H2 (Vddq), U3.H9 (Vddq), U3.K2 (Vdd), U3.K8 (Vdd), U3.N1 (Vdd), U3.N9 (Vdd), U3.R1 (Vdd), U3.R9 (Vdd)
- net DRAM_1_VCORE: now reaches C1.1, C12.1, C15.1, C18.1, C2.1, C20.1, C3.1, C36.1, C38.1, C5.1, C7.1, C9.1, R1.1, U2.A1 (Vddq), U2.A8 (Vddq), U2.B2 (Vdd), U2.C1 (Vddq), U2.C9 (Vddq), U2.D2 (Vddq), U2.D9 (Vdd), U2.E9 (Vddq), U2.F1 (Vddq), U2.G7 (Vdd), U2.H2 (Vddq), U2.H9 (Vddq), U2.K2 (Vdd), U2.K8 (Vdd), U2.N1 (Vdd), U2.N9 (Vdd), U2.R1 (Vdd), U2.R9 (Vdd)
- net SLAVE_EXTvBUS: now reaches U7.10 (EXTVBUS)
- net SLAVE_EXTvBUS: now also U13.3 (~{OC})
- net at C53.1, U7.15 (VDD1.8), U7.26 (VDD1.8): now also C60.1, TP2.1
- net at U7.4 (VBUS): now also R26.2
- net at U6.15 (VDD1.8): now also U6.26 (VDD1.8), C56.1, C59.1
- net at U6.29 (VDDA1.8): now also C57.2
- net at U6.32 (RBIAS): now also R13.2
- net at U6.4 (VBUS): now also R36.2
- net PCIE_REFCLK_P: now reaches U1.Y11 (REFCLKP_D0/-)
- net PCIE_REFCLK_N: now reaches U1.Y12 (REFCLKN_D0/-)
- net VGA_R_0: now reaches U8.4 (A3)
- net VGA_R_0: now also U1.P2 (PL47B/LDQ44/-)
- net VGA_R_1: now reaches U8.5 (A4)
- net VGA_R_1: now also U1.P1 (PL47A/LDQ44/-)
- net VGA_G_0: now reaches U8.6 (A5)
- net VGA_G_0: now also U1.N2 (PL44A/LDQS44/-)
- net VGA_G_1: now reaches U8.7 (A6)
- net VGA_G_1: now also U1.N1 (PL44D/LDQ44/-)
- net VGA_B_0: now reaches U8.8 (A7)
- net VGA_B_0: now also U1.N3 (PL41A/LDQ44/-)
- net VGA_B_1: now reaches U8.9 (A8)
- net VGA_B_1: now also U1.M1 (PL44B/LDQSN44/-)
- net at U1.H6 (VCCIO7/-): now also U1.H7 (VCCIO7/-), U1.J6 (VCCIO7/-)
- net VGA_B_5: now reaches U1.F1 (PL26B/LDQ32/PCLKC6_1)
- net VGA_B_5: now also U10.7 (A6)
- net VGA_G_5: now reaches U1.G1 (PL26D/LDQ32/PCLKC6_0)
- net VGA_G_5: now also U10.5 (A4)
- net VGA_G_4: now reaches U1.G2 (PL26A/LDQ32/PCLKT6_1)
- net VGA_G_4: now also U10.4 (A3)
- net VGA_R_5: now reaches U1.H1 (PL32C/LDQ32/-)
- net VGA_R_5: now also U10.3 (A2)
- net VGA_R_4: now reaches U1.H2 (PL26C/LDQ32/PCLKT6_0)
- net VGA_R_4: now also U10.2 (A1)
- net VGA_B_3: now reaches U1.J1 (PL32B/LDQSN32/-)
- net VGA_B_3: now also U9.7 (A6)
- net VGA_B_4: now reaches U1.J3 (PL29C/LDQ32/GR_PCLK6_1)
- net VGA_B_4: now also U10.6 (A5)
- net VGA_G_3: now reaches U1.K1 (PL32D/LDQ32/-)
- net VGA_G_3: now also U9.5 (A4)
- net VGA_B_2: now reaches U1.K2 (PL32A/LDQS32/-)
- net VGA_B_2: now also U9.6 (A5)
- net VGA_R_3: now reaches U1.L1 (PL44C/LDQ44/-)
- net VGA_R_3: now also U9.3 (A2)
- net VGA_R_2: now reaches U1.L2 (PL41D/LDQ44/-)
- net VGA_R_2: now also U9.2 (A1)
- net VGA_G_2: now reaches U1.L3 (PL41C/LDQ44/-)
- net VGA_G_2: now also U9.4 (A3)
- net at U1.L6 (VCCIO6/-): now also U1.L7 (VCCIO6/-), U1.M6 (VCCIO6/-)
- net FPGA_VCORE: now reaches U1.H10 (VCC/-)
- net FPGA_VCORE: now also U1.H11 (VCC/-), U1.H12 (VCC/-), U1.H13 (VCC/-), U1.H8 (VCC/-), U1.H9 (VCC/-), U1.J13 (VCC/-), U1.J8 (VCC/-), U1.K13 (VCC/-), U1.K8 (VCC/-), U1.L13 (VCC/-), U1.L8 (VCC/-), U1.M13 (VCC/-), U1.M8 (VCC/-), U1.N10 (VCC/-), U1.N11 (VCC/-), U1.N12 (VCC/-), U1.N13 (VCC/-), U1.N8 (VCC/-), U1.N9 (VCC/-)
- net USB_SLAVE_vBUS: now reaches J1.1 (VBUS)
- net USB_SLAVE_vBUS: now also C62.1, R26.1, U13.1 (OUT)
- new net: J3.A10 (+3.3V), J3.A9 (+3.3V), J3.B8 (+3.3V)
- new net: J3.A12 (GND), J3.A15 (GND), J3.A18 (GND), J3.A4 (GND), J3.B13 (GND), J3.B16 (GND), J3.B18 (GND), J3.B4 (GND), J3.B7 (GND)
- new net: J3.A2 (+12V), J3.A3 (+12V), J3.B1 (+12V), J3.B2 (+12V), J3.B3 (+12V)
- new net: R20.1, U13.4 (~{EN})
- new net: J6.A1 (GND), J6.A12 (GND), J6.B1 (GND), J6.B12 (GND)
- new net: J6.A4 (VBUS), J6.A9 (VBUS), J6.B4 (VBUS), J6.B9 (VBUS)
- new net +5V: C61.1, R36.1, U13.5 (IN)
- new net VGA_BUF_HSYNC: R44.2, U8.18 (B1)
- new net VGA_BUF_VSYNC: R45.2, U8.17 (B2)
- no-connect marks 52 -> 61
Other:
- moved on the sheet: J2, R11, R12, R14, R15, R16, R17, R18, R19, R21, R22, R23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
