File: hardware/klein_star_ein/klein_star_ein.kicad_sch (KiCad schematic)
At the start: 140 parts, among them J1 USB_A, J10 AudioJack3_Ground_Switch, J11 AudioJack3_Ground_Switch, J12 AudioJack3_Ground_Switch, J2 DB15_Female_HighDensity_Mount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, J3 Bus_PCI_Express_x1, J4 1367073-1, J5 ARJM11C7-502-AB-ER2-T, J6 USB_C_Receptacle, J7 MEM2051-00-195-00-A, J8 AudioJack3_Ground_Switch, J9 AudioJack3_Ground_Switch, U1 ECP5UM25, U10 SN74ALVC245PWR, U11 KSZ9021RL, U12 TUSB2036, U13 TPS2041B, U2 MT41K512M16, U3 MT41K512M16, U4 FT2232HQ, U5 W25Q128JVS, U6 USB3300-EZK, U7 USB3300-EZK, U8 SN74ALVC245PWR, U9 SN74ALVC245PWR

Commit message: dram layout
Parts:
- removed R1, R6: 0R, Resistor_SMD:R_0603_1608Metric, symbol Device:R_Small
- removed RN8: 51R, Resistor_SMD:R_Array_Concave_4x0402, symbol Device:R_Pack04_Split
- added C66: 470n, Capacitor_SMD:C_0402_1005Metric, symbol Device:C_Small
Connections:
- net +1V35 is gone; now on net 1V35_DRAM_VCORE: U1.H14 (VCCIO2/-), U1.H15 (VCCIO2/-), U1.J15 (VCCIO2/-)
- net DRAM_1_VCORE is gone; now on net 1V35_DRAM_VCORE: C1.1, C12.1, C15.1, C18.1, C2.1, C20.1, C3.1, C36.1, C38.1, C5.1, C7.1, C9.1, U2.A1 (Vddq), U2.A8 (Vddq), U2.B2 (Vdd), U2.C1 (Vddq), U2.C9 (Vddq), U2.D2 (Vddq), U2.D9 (Vdd), U2.E9 (Vddq), U2.F1 (Vddq), U2.G7 (Vdd), U2.H2 (Vddq), U2.H9 (Vddq), U2.K2 (Vdd), U2.K8 (Vdd), U2.N1 (Vdd), U2.N9 (Vdd), U2.R1 (Vdd), U2.R9 (Vdd)
- net DRAM_2_VCORE is gone; now on net 1V35_DRAM_VCORE: C10.1, C13.1, C14.1, C16.1, C17.1, C19.1, C35.1, C37.1, C39.1, C4.1, C6.1, C8.1, U3.A1 (Vddq), U3.A8 (Vddq), U3.B2 (Vdd), U3.C1 (Vddq), U3.C9 (Vddq), U3.D2 (Vddq), U3.D9 (Vdd), U3.E9 (Vddq), U3.F1 (Vddq), U3.G7 (Vdd), U3.H2 (Vddq), U3.H9 (Vddq), U3.K2 (Vdd), U3.K8 (Vdd), U3.N1 (Vdd), U3.N9 (Vdd), U3.R1 (Vdd), U3.R9 (Vdd)
- net DRAM_ADDR_0: now also RN2.6 (R3.2), U1.C17 (PT60B/-); no longer RN2.3 (R3.1)
- net DRAM_ADDR_1: now also RN7.4 (R4.1), U1.B13 (PT42A/-); no longer RN7.3 (R3.1)
- net DRAM_ADDR_10: now also RN7.1 (R1.1), U1.C12 (PT35B/PCLKC1_0)
- net DRAM_ADDR_11: now also RN5.6 (R3.2), U1.C14 (PT47B/-); no longer RN6.1 (R1.1)
- net DRAM_ADDR_12: now also RN7.3 (R3.1), U1.B20 (PT67B/-); no longer RN7.2 (R2.1)
- net DRAM_ADDR_13: now also RN5.8 (R1.2), U1.E13 (PT44B/-); no longer RN1.1 (R1.1)
- net DRAM_ADDR_14: now also RN5.5 (R4.2), U1.A16 (PT56A/-); no longer RN6.4 (R4.1)
- net DRAM_ADDR_15: now also RN7.2 (R2.1), U1.B12 (PT35A/PCLKT1_0)
- net DRAM_ADDR_2: now also RN4.7 (R2.2), U1.D15 (PT53A/-); no longer RN2.1 (R1.1)
- net DRAM_ADDR_3: now also RN2.5 (R4.2), U1.D13 (PT44A/-); no longer RN2.2 (R2.1)
- net DRAM_ADDR_4: now also RN6.2 (R2.1), U1.A14 (PT47A/-); no longer RN7.4 (R4.1)
- net DRAM_ADDR_5: now also RN4.8 (R1.2), U1.C15 (PT51B/-); no longer RN1.4 (R4.1)
- net DRAM_ADDR_6: now also RN6.3 (R3.1), U1.B15 (PT51A/-); no longer RN6.2 (R2.1)
- net DRAM_ADDR_7: now also RN4.6 (R3.2), U1.E14 (PT49B/-); no longer RN1.2 (R2.1)
- net DRAM_ADDR_8: now also RN6.4 (R4.1), U1.C16 (PT58A/-); no longer RN6.3 (R3.1)
- net DRAM_ADDR_9: now also RN5.7 (R2.2), U1.E15 (PT53B/-); no longer RN1.3 (R3.1)
- net DRAM_ADDR_BA0: now also RN2.8 (R1.2), U1.A18 (PT65A/-); no longer RN4.1 (R1.1)
- net DRAM_ADDR_BA1: now also RN6.1 (R1.1), U1.A13 (PT40B/-); no longer RN7.1 (R1.1)
- net DRAM_ADDR_BA2: now also RN2.7 (R2.2), U1.D16 (PT58B/-); no longer RN2.4 (R4.1)
- net DRAM_CKE: now also U1.D11 (PT33A/PCLKT1_1)
- net DRAM_CLK_N: now also U1.E12 (PT38B/GR_PCLK1_1)
- net DRAM_CLK_P: now also U1.D12 (PT38A/GR_PCLK1_0)
- net DRAM_DATA_0: now also U1.J16 (PR11D/RDQ8/-)
- net DRAM_DATA_1: now also U1.G16 (PR8C/RDQ8/-)
- net DRAM_DATA_10: now also U1.F20 (PR17C/RDQ20/-); no longer U1.H5 (PL20C/LDQ20/GR_PCLK7_0)
- net DRAM_DATA_11: now also U1.J20 (PR23C/RDQ20/PCLKT2_0); no longer U1.E1 (PL17D/LDQ20/-)
- net DRAM_DATA_12: now also U1.K19 (PR23B/RDQ20/PCLKC2_1); no longer U1.G3 (PL23A/LDQ20/PCLKT7_1)
- net DRAM_DATA_13: now also U1.J18 (PR20C/RDQ20/GR_PCLK2_0); no longer U1.E2 (PL23D/LDQ20/PCLKC7_0)
- net DRAM_DATA_14: now also U1.K20 (PR23D/RDQ20/PCLKC2_0); no longer U1.F3 (PL23B/LDQ20/PCLKC7_1)
- net DRAM_DATA_15: now also U1.K18 (PR20D/RDQ20/-); no longer U1.F2 (PL23C/LDQ20/PCLKT7_0)
- net DRAM_DATA_16: now also U1.P19 (PR38C/RDQ44/-); no longer U1.F18 (PR5D/RDQ8/-)
- net DRAM_DATA_17: now also U1.U18 (PR47A/RDQ44/-); no longer U1.D18 (PR5A/RDQ8/-)
- net DRAM_DATA_18: now also U1.U20 (PR41D/RDQ44/-); no longer U1.F16 (PR2D/RDQ8/-)
- net DRAM_DATA_19: now also U1.U17 (PR47B/RDQ44/-); no longer U1.D17 (PR2B/RDQ8/S0_IN)
- net DRAM_DATA_2: now also U1.J17 (PR11C/RDQ8/-)
- net DRAM_DATA_20: now also U1.T20 (PR41C/RDQ44/-); no longer U1.G16 (PR8C/RDQ8/-)
- net DRAM_DATA_21: now also U1.U16 (PR47C/RDQ44/LRC_GPLL0T_IN); no longer U1.E16 (PR2C/RDQ8/-)
- net DRAM_DATA_22: now also U1.U19 (PR44C/RDQ44/-); no longer U1.E17 (PR5B/RDQ8/-)
- net DRAM_DATA_23: now also U1.P20 (PR41A/RDQ44/-); no longer U1.E18 (PR5C/RDQ8/-)
- net DRAM_DATA_24: now also U1.R16 (PR35C/RDQ32/-); no longer U1.G20 (PR17D/RDQ20/-)
- net DRAM_DATA_25: now also U1.L17 (PR29B/RDQ32/-); no longer U1.J20 (PR23C/RDQ20/PCLKT2_0)
- net DRAM_DATA_26: now also U1.L18 (PR29C/RDQ32/GR_PCLK3_1); no longer U1.F19 (PR17B/RDQ20/-)
- net DRAM_DATA_27: now also U1.P17 (PR32D/RDQ32/-); no longer U1.K20 (PR23D/RDQ20/PCLKC2_0)
- net DRAM_DATA_28: now also U1.M20 (PR26B/RDQ32/PCLKC3_1); no longer U1.E19 (PR14D/RDQ20/-)
- net DRAM_DATA_29: now also U1.M19 (PR26D/RDQ32/PCLKC3_0); no longer U1.K19 (PR23B/RDQ20/PCLKC2_1)
- net DRAM_DATA_3: now also U1.H16 (PR8D/RDQ8/-)
- net DRAM_DATA_30: now also U1.M18 (PR29D/RDQ32/-); no longer U1.D19 (PR14B/RDQ20/-)
- net DRAM_DATA_31: now also U1.N18 (PR32C/RDQ32/-); no longer U1.J19 (PR23A/RDQ20/PCLKT2_1)
- net DRAM_DATA_4: now also U1.C18 (PR2A/RDQ8/-); no longer U1.B4 (PL5B/LDQ8/-)
- net DRAM_DATA_5: now also U1.E18 (PR5C/RDQ8/-); no longer U1.C4 (PL5A/LDQ8/-)
- net DRAM_DATA_6: now also U1.D17 (PR2B/RDQ8/S0_IN); no longer U1.B3 (PL5D/LDQ8/-)
- net DRAM_DATA_7: now also U1.D18 (PR5A/RDQ8/-); no longer U1.C5 (PL2D/LDQ8/-)
- net DRAM_DATA_8: now also U1.F19 (PR17B/RDQ20/-); no longer U1.H3 (PL20D/LDQ20/-)
- net DRAM_DATA_9: now also U1.J19 (PR23A/RDQ20/PCLKT2_1)
- net DRAM_DM0: now also U1.H17 (PR11B/RDQ8/-)
- net DRAM_DM1: now also U1.E19 (PR14D/RDQ20/-)
- net DRAM_DM2: now also U1.T17 (PR47D/RDQ44/LRC_GPLL0C_IN); no longer U1.C18 (PR2A/RDQ8/-)
- net DRAM_DM3: now also U1.R17 (PR35D/RDQ32/-); no longer U1.J18 (PR20C/RDQ20/GR_PCLK2_0)
- net DRAM_DQS0_N: now also U1.G18 (PR8B/RDQSN8/-); no longer U1.D5 (PL8B/LDQSN8/-)
- net DRAM_DQS0_P: now also U1.F17 (PR8A/RDQS8/-); no longer U1.E4 (PL8A/LDQS8/-)
- net DRAM_DQS1_N: now also U1.H20 (PR20B/RDQSN20/-); no longer U1.G5 (PL20B/LDQSN20/-)
- net DRAM_DQS1_P: now also U1.G19 (PR20A/RDQS20/GR_PCLK2_1); no longer U1.H4 (PL20A/LDQS20/GR_PCLK7_1)
- net DRAM_DQS2_N: now also U1.R18 (PR44B/RDQSN44/-); no longer U1.G18 (PR8B/RDQSN8/-)
- net DRAM_DQS2_P: now also U1.T19 (PR44A/RDQS44/-); no longer U1.F17 (PR8A/RDQS8/-)
- net DRAM_DQS3_N: now also U1.M17 (PR32B/RDQSN32/-); no longer U1.H20 (PR20B/RDQSN20/-)
- net DRAM_DQS3_P: now also U1.N16 (PR32A/RDQS32/-); no longer U1.G19 (PR20A/RDQS20/GR_PCLK2_1)
- net DRAM_ODT: now also RN1.6 (R3.2); no longer RN4.4 (R4.1)
- net DRAM_VREF: now also U1.D20 (PR14C/RDQ20/VREF1_2), U1.P16 (PR35B/RDQ32/VREF1_3)
- net DRAM_nCAS: now also RN1.7 (R2.2), U1.A19 (PT67A/-); no longer RN5.1 (R1.1)
- net DRAM_nCS: now also RN1.5 (R4.2), U1.B19 (PT65B/-); no longer RN4.2 (R2.1)
- net DRAM_nRAS: now also RN1.8 (R1.2), U1.A17 (PT62A/-); no longer RN5.2 (R2.1)
- net DRAM_nRESET: now also U1.D14 (PT49A/-)
- net DRAM_nWE: now also U1.A12 (PT40A/-); no longer RN4.3 (R3.1)
- net GND: now also RN1.1 (R1.1), RN1.2 (R2.1), RN1.3 (R3.1), RN1.4 (R4.1), RN2.1 (R1.1), RN2.2 (R2.1), RN2.3 (R3.1), RN2.4 (R4.1), RN4.1 (R1.1), RN4.2 (R2.1), RN4.3 (R3.1), RN5.1 (R1.1), RN5.2 (R2.1), RN5.3 (R3.1), RN5.4 (R4.1), C66.2; no longer RN1.5 (R4.2), RN1.6 (R3.2), RN1.7 (R2.2), RN1.8 (R1.2), RN2.5 (R4.2), RN2.6 (R3.2), RN2.7 (R2.2), RN2.8 (R1.2), RN4.5 (R4.2), RN4.6 (R3.2), RN4.7 (R2.2), RN4.8 (R1.2), RN5.7 (R2.2), RN5.8 (R1.2)
- net 1V35_DRAM_VCORE: now reaches U1.F11 (VCCIO1/-)
- net 1V35_DRAM_VCORE: now also U1.F12 (VCCIO1/-), U1.L14 (VCCIO3/-), U1.L15 (VCCIO3/-), U1.M15 (VCCIO3/-), C66.1
- now unconnected: U1.B16 (PT56B/-), U1.B17 (PT60A/-), U1.B18 (PT62B/-), U1.C13 (PT42B/-), U1.E11 (PT33B/PCLKC1_1)
- no-connect marks 87 -> 78
Other:
- moved on the sheet: U1B, U1D, U1F
