File: hardware/klein_star_ein/klein_star_ein.kicad_sch (KiCad schematic)
At the start: 138 parts, among them J1 USB_A, J10 AudioJack3_Ground_Switch, J11 AudioJack3_Ground_Switch, J12 AudioJack3_Ground_Switch, J2 DB15_Female_HighDensity_Mount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, J3 Bus_PCI_Express_x1, J4 1367073-1, J5 ARJM11C7-502-AB-ER2-T, J6 USB_C_Receptacle, J7 MEM2051-00-195-00-A, J8 AudioJack3_Ground_Switch, J9 AudioJack3_Ground_Switch, U1 ECP5UM25, U10 SN74ALVC245PWR, U11 KSZ9021RL, U12 TUSB2036, U13 TPS2041B, U2 MT41K512M16, U3 MT41K512M16, U4 FT2232HQ, U5 W25Q128JVS, U6 USB3300-EZK, U7 USB3300-EZK, U8 SN74ALVC245PWR, U9 SN74ALVC245PWR

Commit message: rzeczy
Parts:
- removed RN6: 51R, Resistor_SMD:R_Array_Concave_4x0402, symbol Device:R_Pack04_Split
- removed RN7: 51R, symbol Device:R_Pack04_Split
- added C67: 100n, Capacitor_SMD:C_0603_1608Metric, symbol Device:C_Small
- added J13: Conn_01x05, Connector_PinHeader_2.54mm:PinHeader_1x05_P2.54mm_Vertical, symbol Connector_Generic:Conn_01x05
- C43, C44, C45, C46, C48, C49, C50, C51, C53, C54, C56, C57, C59, C60: footprint Capacitor_SMD:C_0402_1005Metric -> Capacitor_SMD:C_0603_1608Metric
- C47, C52: value 4u7 -> 100nF; footprint Capacitor_SMD:C_0402_1005Metric -> Capacitor_SMD:C_0603_1608Metric
- R20: footprint Resistor_SMD:R_0402_1005Metric_Pad0.72x0.64mm_HandSolder -> Resistor_SMD:R_0603_1608Metric
Connections:
- net +3V3: now also U1.L6 (VCCIO6/-), U1.L7 (VCCIO6/-), U1.M6 (VCCIO6/-), C67.1
- net DRAM_ADDR_0: now also RN5.6 (R3.2), U1.B17 (PT60A/-); no longer RN2.6 (R3.2), U1.C17 (PT60B/-)
- net DRAM_ADDR_1: now also U1.C13 (PT42B/-); no longer U1.B13 (PT42A/-)
- net DRAM_ADDR_10: now also U1.D16 (PT58B/-); no longer U1.C12 (PT35B/PCLKC1_0)
- net DRAM_ADDR_11: now also RN2.8 (R1.2), U1.A18 (PT65A/-); no longer RN5.6 (R3.2), U1.C14 (PT47B/-)
- net DRAM_ADDR_13: now also RN1.6 (R3.2), U1.A14 (PT47A/-); no longer RN5.8 (R1.2), U1.E13 (PT44B/-)
- net DRAM_ADDR_14: now also RN2.7 (R2.2), U1.D11 (PT33A/PCLKT1_1); no longer RN5.5 (R4.2), U1.A16 (PT56A/-)
- net DRAM_ADDR_15: now also RN5.7 (R2.2), U1.C15 (PT51B/-); no longer U1.B12 (PT35A/PCLKT1_0)
- net DRAM_ADDR_2: now also RN1.8 (R1.2), U1.B16 (PT56B/-); no longer RN4.7 (R2.2), U1.D15 (PT53A/-)
- net DRAM_ADDR_3: now also RN5.8 (R1.2), U1.A17 (PT62A/-); no longer RN2.5 (R4.2), U1.D13 (PT44A/-)
- net DRAM_ADDR_4: now also U1.C14 (PT47B/-); no longer U1.A14 (PT47A/-)
- net DRAM_ADDR_5: now also U1.A16 (PT56A/-); no longer RN4.8 (R1.2), U1.C15 (PT51B/-)
- net DRAM_ADDR_6: now also RN2.5 (R4.2), U1.E11 (PT33B/PCLKC1_1); no longer U1.B15 (PT51A/-)
- net DRAM_ADDR_7: now also RN1.7 (R2.2), U1.A13 (PT40B/-); no longer RN4.6 (R3.2), U1.E14 (PT49B/-)
- net DRAM_ADDR_8: now also RN2.6 (R3.2), U1.C12 (PT35B/PCLKC1_0); no longer U1.C16 (PT58A/-)
- net DRAM_ADDR_9: now also RN1.5 (R4.2), U1.B15 (PT51A/-); no longer RN5.7 (R2.2), U1.E15 (PT53B/-)
- net DRAM_ADDR_BA0: now also RN5.5 (R4.2), U1.A12 (PT40A/-); no longer RN2.8 (R1.2), U1.A18 (PT65A/-)
- net DRAM_ADDR_BA1: now also U1.E15 (PT53B/-); no longer U1.A13 (PT40B/-)
- net DRAM_ADDR_BA2: now also RN4.5 (R4.2), U1.B12 (PT35A/PCLKT1_0); no longer RN2.7 (R2.2), U1.D16 (PT58B/-)
- net DRAM_CKE: now also U1.D13 (PT44A/-); no longer U1.D11 (PT33A/PCLKT1_1)
- net DRAM_DATA_0: now also U1.K20 (PR23D/RDQ20/PCLKC2_0); no longer U1.J16 (PR11D/RDQ8/-)
- net DRAM_DATA_1: now also U1.F20 (PR17C/RDQ20/-); no longer U1.G16 (PR8C/RDQ8/-)
- net DRAM_DATA_10: now also U1.F18 (PR5D/RDQ8/-); no longer U1.F20 (PR17C/RDQ20/-)
- net DRAM_DATA_11: now also U1.H16 (PR8D/RDQ8/-); no longer U1.J20 (PR23C/RDQ20/PCLKT2_0)
- net DRAM_DATA_12: now also U1.F16 (PR2D/RDQ8/-); no longer U1.K19 (PR23B/RDQ20/PCLKC2_1)
- net DRAM_DATA_13: now also U1.J17 (PR11C/RDQ8/-); no longer U1.J18 (PR20C/RDQ20/GR_PCLK2_0)
- net DRAM_DATA_14: now also U1.E16 (PR2C/RDQ8/-); no longer U1.K20 (PR23D/RDQ20/PCLKC2_0)
- net DRAM_DATA_15: now also U1.J16 (PR11D/RDQ8/-); no longer U1.K18 (PR20D/RDQ20/-)
- net DRAM_DATA_16: now also U1.N17 (PR35A/RDQ32/-); no longer U1.P19 (PR38C/RDQ44/-)
- net DRAM_DATA_17: now also U1.L17 (PR29B/RDQ32/-); no longer U1.U18 (PR47A/RDQ44/-)
- net DRAM_DATA_18: now also U1.R17 (PR35D/RDQ32/-); no longer U1.U20 (PR41D/RDQ44/-)
- net DRAM_DATA_19: now also U1.M18 (PR29D/RDQ32/-); no longer U1.U17 (PR47B/RDQ44/-)
- net DRAM_DATA_2: now also U1.J20 (PR23C/RDQ20/PCLKT2_0); no longer U1.J17 (PR11C/RDQ8/-)
- net DRAM_DATA_20: now also U1.P17 (PR32D/RDQ32/-); no longer U1.T20 (PR41C/RDQ44/-)
- net DRAM_DATA_21: now also U1.N18 (PR32C/RDQ32/-); no longer U1.U16 (PR47C/RDQ44/LRC_GPLL0T_IN)
- net DRAM_DATA_22: now also U1.R16 (PR35C/RDQ32/-); no longer U1.U19 (PR44C/RDQ44/-)
- net DRAM_DATA_23: now also U1.L16 (PR29A/RDQ32/GR_PCLK3_0); no longer U1.P20 (PR41A/RDQ44/-)
- net DRAM_DATA_24: now also U1.P20 (PR41A/RDQ44/-); no longer U1.R16 (PR35C/RDQ32/-)
- net DRAM_DATA_25: now also U1.U20 (PR41D/RDQ44/-); no longer U1.L17 (PR29B/RDQ32/-)
- net DRAM_DATA_26: now also U1.N19 (PR38A/RDQ44/-); no longer U1.L18 (PR29C/RDQ32/GR_PCLK3_1)
- net DRAM_DATA_27: now also U1.U19 (PR44C/RDQ44/-); no longer U1.P17 (PR32D/RDQ32/-)
- net DRAM_DATA_28: now also U1.P19 (PR38C/RDQ44/-); no longer U1.M20 (PR26B/RDQ32/PCLKC3_1)
- net DRAM_DATA_29: now also U1.T18 (PR44D/RDQ44/-); no longer U1.M19 (PR26D/RDQ32/PCLKC3_0)
- net DRAM_DATA_3: now also U1.F19 (PR17B/RDQ20/-); no longer U1.H16 (PR8D/RDQ8/-)
- net DRAM_DATA_30: now also U1.N20 (PR38B/RDQ44/-); no longer U1.M18 (PR29D/RDQ32/-)
- net DRAM_DATA_31: now also U1.T20 (PR41C/RDQ44/-); no longer U1.N18 (PR32C/RDQ32/-)
- net DRAM_DATA_4: now also U1.D19 (PR14B/RDQ20/-); no longer U1.C18 (PR2A/RDQ8/-)
- net DRAM_DATA_5: now also U1.E20 (PR17A/RDQ20/-); no longer U1.E18 (PR5C/RDQ8/-)
- net DRAM_DATA_6: now also U1.J19 (PR23A/RDQ20/PCLKT2_1); no longer U1.D17 (PR2B/RDQ8/S0_IN)
- net DRAM_DATA_7: now also U1.C20 (PR14A/RDQ20/-); no longer U1.D18 (PR5A/RDQ8/-)
- net DRAM_DATA_8: now also U1.E18 (PR5C/RDQ8/-); no longer U1.F19 (PR17B/RDQ20/-)
- net DRAM_DATA_9: now also U1.G16 (PR8C/RDQ8/-); no longer U1.J19 (PR23A/RDQ20/PCLKT2_1)
- net DRAM_DM0: now also U1.G20 (PR17D/RDQ20/-); no longer U1.H17 (PR11B/RDQ8/-)
- net DRAM_DM1: now also U1.E17 (PR5B/RDQ8/-); no longer U1.E19 (PR14D/RDQ20/-)
- net DRAM_DM2: now also U1.M20 (PR26B/RDQ32/PCLKC3_1); no longer U1.T17 (PR47D/RDQ44/LRC_GPLL0C_IN)
- net DRAM_DM3: now also U1.U18 (PR47A/RDQ44/-); no longer U1.R17 (PR35D/RDQ32/-)
- net DRAM_DQS0_N: now also U1.H20 (PR20B/RDQSN20/-); no longer U1.G18 (PR8B/RDQSN8/-)
- net DRAM_DQS0_P: now also U1.G19 (PR20A/RDQS20/GR_PCLK2_1); no longer U1.F17 (PR8A/RDQS8/-)
- net DRAM_DQS1_N: now also U1.G18 (PR8B/RDQSN8/-); no longer U1.H20 (PR20B/RDQSN20/-)
- net DRAM_DQS1_P: now also U1.F17 (PR8A/RDQS8/-); no longer U1.G19 (PR20A/RDQS20/GR_PCLK2_1)
- net DRAM_DQS2_N: now also U1.M17 (PR32B/RDQSN32/-); no longer U1.R18 (PR44B/RDQSN44/-)
- net DRAM_DQS2_P: now also U1.N16 (PR32A/RDQS32/-); no longer U1.T19 (PR44A/RDQS44/-)
- net DRAM_DQS3_N: now also U1.R18 (PR44B/RDQSN44/-); no longer U1.M17 (PR32B/RDQSN32/-)
- net DRAM_DQS3_P: now also U1.T19 (PR44A/RDQS44/-); no longer U1.N16 (PR32A/RDQS32/-)
- net DRAM_ODT: now also RN4.8 (R1.2), U1.C17 (PT60B/-); no longer RN1.6 (R3.2)
- net DRAM_nCAS: now also U1.C16 (PT58A/-); no longer RN1.7 (R2.2), U1.A19 (PT67A/-)
- net DRAM_nCS: now also RN4.7 (R2.2), U1.D14 (PT49A/-); no longer RN1.5 (R4.2), U1.B19 (PT65B/-)
- net DRAM_nRAS: now also U1.D15 (PT53A/-); no longer RN1.8 (R1.2), U1.A17 (PT62A/-)
- net DRAM_nRESET: now also U1.B13 (PT42A/-); no longer U1.D14 (PT49A/-)
- net DRAM_nWE: now also RN4.6 (R3.2), U1.A19 (PT67A/-); no longer U1.A12 (PT40A/-)
- net FIFO_D0/RX: now also U1.L2 (PL41D/LDQ44/-)
- net FIFO_D1/TX: now also U1.L1 (PL44C/LDQ44/-)
- net FIFO_D2: now also U1.K2 (PL32A/LDQS32/-)
- net FIFO_D3: now also U1.K1 (PL32D/LDQ32/-)
- net FIFO_D4: now also U1.L3 (PL41C/LDQ44/-)
- net FIFO_D5: now also U1.J1 (PL32B/LDQSN32/-)
- net FIFO_D6: now also U1.H2 (PL26C/LDQ32/PCLKT6_0)
- net FIFO_D7: now also U1.H1 (PL32C/LDQ32/-)
- net FIFO_WKUP: now also U1.F1 (PL26B/LDQ32/PCLKC6_1)
- net FIFO_nRD: now also U1.J4 (PL29A/LDQ32/GR_PCLK6_0)
- net FIFO_nRXE: now also U1.G2 (PL26A/LDQ32/PCLKT6_1)
- net FIFO_nTXE: now also U1.G1 (PL26D/LDQ32/PCLKC6_0)
- net FIFO_nWR: now also U1.J3 (PL29C/LDQ32/GR_PCLK6_1)
- net GND: now also C54.2, C57.2, J6.A1 (GND), J6.A12 (GND), J6.B1 (GND), J6.B12 (GND), J6.S1 (SHIELD), J7.3 (VSS), RN4.4 (R4.1), C67.2, J13.5 (Pin_5); no longer C54.1, C57.1, U12.28 (GND), U12.7 (GND)
- net JTAG_TCK: now also U1.T5 (TCK/-), J13.1 (Pin_1)
- net JTAG_TDI: now also U1.R5 (TDI/-), J13.2 (Pin_2)
- net JTAG_TDO: now also U1.V4 (TDO/-), J13.3 (Pin_3)
- net JTAG_TMS: now also U1.U5 (TMS/-), J13.4 (Pin_4)
- net USB_HOST_DATA0: now also U1.A6 (PT4A/-)
- net USB_HOST_DATA1: now also U1.B6 (PT4B/-)
- net USB_HOST_DATA2: now also U1.A5 (PL2B/LDQ8/-)
- net USB_HOST_DATA3: now also U1.B5 (PL2C/LDQ8/-)
- net USB_HOST_DATA4: now also U1.A4 (PL2A/LDQ8/-)
- net USB_HOST_DATA5: now also U1.B4 (PL5B/LDQ8/-)
- net USB_HOST_DATA6: now also U1.A3 (PL5C/LDQ8/-)
- net USB_HOST_DATA7: now also U1.B3 (PL5D/LDQ8/-)
- net USB_SLAVE_CLK: now also U1.A11 (PT27B/PCLKC0_1)
- net USB_SLAVE_CLKOUT: now also U1.C8 (PT15A/-)
- net USB_SLAVE_DATA0: now also U1.C11 (PT29B/PCLKC0_0)
- net USB_SLAVE_DATA1: now also U1.B11 (PT29A/PCLKT0_0)
- net USB_SLAVE_DATA2: now also U1.C10 (PT22B/-)
- net USB_SLAVE_DATA3: now also U1.B10 (PT24B/GR_PCLK0_0)
- net USB_SLAVE_DATA4: now also U1.E9 (PT20B/-)
- net USB_SLAVE_DATA5: now also U1.E8 (PT13A/-)
- net USB_SLAVE_DATA6: now also U1.E7 (PT9A/-)
- net USB_SLAVE_DATA7: now also U1.D8 (PT13B/-)
- net USB_SLAVE_DIR: now also U1.D7 (PT9B/-)
- net USB_SLAVE_NXT: now also U1.C7 (PT11B/-)
- net USB_SLAVE_RESET: now also U1.C6 (PT11A/-)
- net USB_SLAVE_STP: now also U1.E6 (PT6A/-)
- net VGA_B_0: now also U10.4 (A3); no longer U1.N3 (PL41A/LDQ44/-), U8.8 (A7)
- net VGA_B_1: now also U1.K3 (PL29D/LDQ32/-), U10.5 (A4); no longer U1.M1 (PL44B/LDQSN44/-), U8.9 (A8)
- net VGA_B_2: now also U1.L4 (PL35C/LDQ32/-), U10.6 (A5); no longer U1.K2 (PL32A/LDQS32/-), U9.6 (A5)
- net VGA_B_3: now also U1.K4 (PL35A/LDQ32/-), U10.7 (A6); no longer U1.J1 (PL32B/LDQSN32/-), U9.7 (A6)
- net VGA_B_4: now also U1.K5 (PL35B/LDQ32/VREF1_6), U10.8 (A7); no longer U1.J3 (PL29C/LDQ32/GR_PCLK6_1), U10.6 (A5)
- net VGA_B_5: now also U1.J5 (PL29B/LDQ32/-), U10.9 (A8); no longer U1.F1 (PL26B/LDQ32/PCLKC6_1), U10.7 (A6)
- net VGA_G_0: now also U1.M1 (PL44B/LDQSN44/-), U9.4 (A3); no longer U1.N2 (PL44A/LDQS44/-), U8.6 (A5)
- net VGA_G_1: now also U1.N3 (PL41A/LDQ44/-), U9.5 (A4); no longer U1.N1 (PL44D/LDQ44/-), U8.7 (A6)
- net VGA_G_2: now also U1.N4 (PL38C/LDQ44/-), U9.6 (A5); no longer U1.L3 (PL41C/LDQ44/-), U9.4 (A3)
- net VGA_G_3: now also U1.M3 (PL41B/LDQ44/-), U9.7 (A6); no longer U1.K1 (PL32D/LDQ32/-), U9.5 (A4)
- net VGA_G_4: now also U1.M4 (PL38A/LDQ44/-), U9.8 (A7); no longer U1.G2 (PL26A/LDQ32/PCLKT6_1), U10.4 (A3)
- net VGA_G_5: now also U1.L5 (PL35D/LDQ32/-), U9.9 (A8); no longer U1.G1 (PL26D/LDQ32/PCLKC6_0), U10.5 (A4)
- net VGA_HSYNC: now also U1.N2 (PL44A/LDQS44/-); no longer U1.P4 (PL47D/LDQ44/LLC_GPLL0C_IN)
- net VGA_R_0: now also U1.N5 (PL38B/LDQ44/-); no longer U1.P2 (PL47B/LDQ44/-)
- net VGA_R_1: now also U1.P5 (PL38D/LDQ44/-); no longer U1.P1 (PL47A/LDQ44/-)
- net VGA_R_2: now also U1.P4 (PL47D/LDQ44/LLC_GPLL0C_IN), U8.6 (A5); no longer U1.L2 (PL41D/LDQ44/-), U9.2 (A1)
- net VGA_R_3: now also U1.P3 (PL47C/LDQ44/LLC_GPLL0T_IN), U8.7 (A6); no longer U1.L1 (PL44C/LDQ44/-), U9.3 (A2)
- net VGA_R_4: now also U1.P2 (PL47B/LDQ44/-), U8.8 (A7); no longer U1.H2 (PL26C/LDQ32/PCLKT6_0), U10.2 (A1)
- net VGA_R_5: now also U1.P1 (PL47A/LDQ44/-), U8.9 (A8); no longer U1.H1 (PL32C/LDQ32/-), U10.3 (A2)
- net VGA_VSYNC: now also U1.N1 (PL44D/LDQ44/-); no longer U1.P3 (PL47C/LDQ44/LLC_GPLL0T_IN)
- net SD_DATA1: now reaches J7.1 (DAT1)
- net SD_DATA1: now also U1.A7 (PT18A/-)
- net SD_DATA0: now reaches J7.2 (DAT0)
- net SD_DATA0: now also U1.A8 (PT18B/-)
- net SD_CLK: now reaches J7.4 (CLK)
- net SD_CLK: now also U1.B8 (PT15B/-)
- net SD_CMD: now reaches J7.6 (CMD)
- net SD_CMD: now also U1.A9 (PT24A/GR_PCLK0_1)
- net SD_DATA3: now reaches J7.7 (CD/DAT3)
- net SD_DATA3: now also U1.B9 (PT22A/-)
- net SD_DATA2: now reaches J7.8 (DAT2)
- net SD_DATA2: now also U1.A10 (PT27A/PCLKT0_1)
- net at U12.1 (DP0): now also J6.A6 (D+), J6.B6 (D+)
- net at U12.2 (DM0): now also J6.A7 (D-), J6.B7 (D-)
- net at U6.29 (VDDA1.8): now also C59.1; no longer C57.2
- net at C53.1, TP2.1, U7.15 (VDD1.8)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: now also C54.1; no longer C60.1
- net at U7.29 (VDDA1.8): now also C60.1; no longer C54.2
- net at C56.1, U6.15 (VDD1.8), U6.26 (VDD1.8): now also C57.1; no longer C59.1
- net 5V_USB: now reaches J6.A4 (VBUS), J6.A9 (VBUS), J6.B4 (VBUS), J6.B9 (VBUS)
- now unconnected: U1.D6 (PT6B/-), U1.D9 (PT20A/-)
- no-connect marks 78 -> 100
Other:
- note added: "REACHABLE"
- note added: "REACHABLE, 1V35"
- moved on the sheet: J6, J7, U12, U1A

Commit message: merge power
Parts:
- added C68, C69, C70, C71, C72, C73, C74, C75, C76, C77, C78, C79, C80, C81, C82, C83, C84, C85, C86: 0.1uF, Capacitor_SMD:C_0603_1608Metric, symbol Device:C
- added R1, R3: R220, Resistor_SMD:R_0402_1005Metric_Pad0.72x0.64mm_HandSolder, symbol Device:R
Connections:
- net +3V3: now also U11.16 (AVDDH), U11.20 (DVDDH), U11.30 (DVDDH), U11.37 (DVDDH), U11.44 (DVDDH), U11.6 (AVDDH), U11.61 (AVDDH), U11.64 (AVDDH), C68.1, C69.1, C70.1, C71.2, C77.1, C78.1, C79.1, C80.2, R1.2, R3.1
- net GND: now also J5.S1 (SHIELD), J5.S2 (SHIELD), C68.2, C69.2, C70.2, C71.1, C72.1, C73.2, C74.2, C75.2, C76.1, C77.2, C78.2, C79.2, C80.1, C81.1, C82.1, C83.2, C84.2, C85.2, C86.1
- net +1V2: now reaches U11.12 (AVDDL)
- net +1V2: now also U11.13 (AVDDL), U11.22 (DVDDL), U11.29 (DVDDL), U11.35 (DVDDL), U11.4 (AVDDL), U11.40 (DVDDL), U11.5 (AVDDL), U11.52 (DVDDL), U11.54 (DVDDL), U11.58 (AVDD_PLL), C72.2, C73.1, C74.1, C75.1, C76.2, C81.2, C82.2, C83.1, C84.1, C85.1, C86.2
- net at U11.19 (LED2/PHYAD1): now also J5.L2 (LED-L_K_GRN)
- net at U11.21 (LED1/PHYAD0): now also J5.L4 (LED-R_K_YLW)
- net TX0: now reaches U11.24 (TXD0)
- net TX1: now reaches U11.25 (TXD1)
- net TX2: now reaches U11.26 (TXD2)
- net TX3: now reaches U11.27 (TXD3)
- net TX_CLK: now reaches U11.32 (GTX_CLK)
- net TX_CTRL: now reaches U11.33 (TX_EN)
- net RX3: now reaches U11.36 (RXD3/MODE3)
- net RX2: now reaches U11.38 (RXD2/MODE2)
- net RX1: now reaches U11.41 (RXD1/MODE1)
- net RX0: now reaches U11.42 (RXD0/MODE0)
- net RX_CTRL: now reaches U11.43 (RX_DV/CLK125_EN)
- net RX_CLK: now reaches U11.46 (RX_CLK/PHYAD2)
- net MDC: now reaches U11.48 (MDC)
- net MDIO: now reaches U11.49 (MDIO)
- net INT: now reaches U11.51 (INT_N)
- net CLK125: now reaches U11.55 (CLK125_NDO/LED_MODE)
- net RESET: now reaches U11.56 (nRESET)
- net at J5.L1 (LED-L_A_GRN): now also R1.1
- net at J5.L3 (LED-R_A_YLW): now also R3.2
- no-connect marks 100 -> 101
Other:
- added sheet Power_converter_1V2 (Power_converter.kicad_sch)
- added sheet Power_converter_1V2_FPGA (Power_converter.kicad_sch)
- added sheet Power_converter_1V35 (Power_converter.kicad_sch)
- added sheet Power_converter_2V5 (Power_converter.kicad_sch)
- added sheet Power_converter_3V3 (Power_converter.kicad_sch)
- note added: "Resistor values: 1V2 FPGA: 200k - 200k 1V2: 200k - 200k 3V3: 200k - 44.2k 2V5: 200k - 63.2k 1V35 VRAM: 200k - 160k"
- note added: "TODO: ISET and XO XI pins"
- note added: "TODO: TRCT pins"
