File: hardware/klein_star_ein/klein_star_ein.kicad_pcb (KiCad board)
At the start: 6 copper layers, 100 x 90 mm, 138 parts, among them J1 USB_A, J10 AudioJack3_Ground_Switch, J11 AudioJack3_Ground_Switch, J12 AudioJack3_Ground_Switch, J2 DB15_Female_HighDensity_Mount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, J3 Bus_PCI_Express_x1, J4 1367073-1, J5 ARJM11C7-502-AB-ER2-T, J6 USB_C_Receptacle, J7 MEM2051-00-195-00-A, J8 AudioJack3_Ground_Switch, J9 AudioJack3_Ground_Switch, U1 ECP5UM25, U10 SN74ALVC245PWR, U11 KSZ9021RL, U12 TUSB2036, U13 TPS2041B, U2 MT41K512M16, U3 MT41K512M16, U4 FT2232HQ, U5 W25Q128JVS, U6 USB3300-EZK, U7 USB3300-EZK, U8 SN74ALVC245PWR, U9 SN74ALVC245PWR

Commit message: what the fuck
Parts:
- C11, C13, C39, C40, C41, C42, C55, C8, R79, R80: moved to F.Cu
- moved C2 84.8 mm to (235.6, 157.3), turned to 0 degrees
- moved C16 80.6 mm to (238.5, 153.7), turned to 0 degrees
- moved C9 79.5 mm to (232.7, 155.3), turned to 0 degrees
- moved C1 78.7 mm to (229.8, 153.8), turned to 0 degrees
- moved C7 75.2 mm to (229.8, 155.8), turned to 0 degrees
- moved C55 75.1 mm to (238.5, 155.7), turned to 0 degrees
- moved C12 73.5 mm to (235.6, 155.3), turned to 0 degrees
- moved C41 72.3 mm to (235.6, 153.3)
- moved C38 71.4 mm to (224.1, 157.7), turned to 0 degrees
- moved C11 71.2 mm to (229.8, 159.7), turned to 0 degrees
- moved R2 70.9 mm to (218.3, 160.9), turned to 0 degrees
- moved C13 68.5 mm to (227.0, 157.7), turned to 0 degrees
- moved C3 68.2 mm to (232.7, 157.3), turned to 0 degrees
- moved C17 67.7 mm to (224.1, 153.8), turned to 0 degrees
- moved C5 67.0 mm to (227.0, 153.8), turned to 0 degrees
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Routing:
- net GND: track 278.7 -> 107.3 mm, vias 79 -> 27
- net 1V35_DRAM_VCORE: track 104.0 -> 8.20 mm, vias 44 -> 6
- net /DRAM_ADDR_10: track 78.6 -> 0.00 mm, vias 3 -> 0
- net /DRAM_ADDR_15: track 77.6 -> 0.00 mm, vias 3 -> 0
- net /DRAM_ADDR_8: track 76.6 -> 0.00 mm, vias 3 -> 0
- net /DRAM_ADDR_BA1: track 76.6 -> 0.00 mm, vias 3 -> 0
- net /DRAM_ADDR_4: track 76.5 -> 0.00 mm, vias 3 -> 0
- net /DRAM_ADDR_2: track 76.5 -> 0.00 mm, vias 4 -> 0
- net /DRAM_ADDR_11: track 75.9 -> 0.00 mm, vias 3 -> 0
- net /DRAM_ADDR_6: track 75.5 -> 0.00 mm, vias 3 -> 0
- net /DRAM_nCS: track 75.5 -> 0.00 mm, vias 4 -> 0
- net /DRAM_ADDR_0: track 75.1 -> 0.00 mm, vias 4 -> 0
- net /DRAM_nCAS: track 75.0 -> 0.00 mm, vias 4 -> 0
- net /DRAM_ADDR_14: track 74.7 -> 0.00 mm, vias 3 -> 0
- net /DRAM_ADDR_BA2: track 74.7 -> 0.00 mm, vias 3 -> 0
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- removed copper zone on In3.Cu, net 1V35_DRAM_VCORE

Commit message: rzeczy
Parts:
- removed RN6, RN7: 51R, Resistor_SMD:R_Array_Concave_4x0402
- added C67: 100n, Capacitor_SMD:C_0603_1608Metric, F.Cu at (134.1, 133.4)
- added J13: Conn_01x05, Connector_PinHeader_2.54mm:PinHeader_1x05_P2.54mm_Vertical, F.Cu at (123.6, 140.6)
- added kibuzzard-61F2DE20: G***, kibuzzard-61F2DE20, F.Cu at (148.0, 117.2)
- added kibuzzard-61F2DE36: G***, kibuzzard-61F2DE36, F.Cu at (168.5, 126.6)
- added kibuzzard-61F2DE40: G***, kibuzzard-61F2DE40, F.Cu at (168.5, 129.0)
- added kibuzzard-61F2DEBF: G***, kibuzzard-61F2DEBF, F.Cu at (187.9, 132.8)
- added kibuzzard-61F30A02: G***, kibuzzard-61F30A02, F.Cu at (128.2, 133.8)
- added kibuzzard-61F30A12: G***, kibuzzard-61F30A12, F.Cu at (113.2, 126.1)
- added kibuzzard-61F30A21: G***, kibuzzard-61F30A21, F.Cu at (124.6, 143.4)
- added kibuzzard-61F31B82: G***, kibuzzard-61F31B82, F.Cu at (158.2, 94.0)
- added kibuzzard-61F31C80: G***, kibuzzard-61F31C80, F.Cu at (171.1, 105.9)
- added kibuzzard-61F32E72: G***, kibuzzard-61F32E72, F.Cu at (142.3, 94.0)
- C11, C40, C42, C55, R79, R80: moved to B.Cu
- C27, C31, C32, C33, C34, L1, L2: moved to F.Cu
- C43, C44, C45, C46, C48, C49, C50, C51, C53, C54, C56, C57, C59, C60: footprint Capacitor_SMD:C_0402_1005Metric -> Capacitor_SMD:C_0603_1608Metric
- C47, C52: value 4u7 -> 100nF; footprint Capacitor_SMD:C_0402_1005Metric -> Capacitor_SMD:C_0603_1608Metric
- R20: footprint Resistor_SMD:R_0402_1005Metric_Pad0.72x0.64mm_HandSolder -> Resistor_SMD:R_0603_1608Metric
- moved R106 93.4 mm to (160.6, 96.2), turned to 0 degrees
- moved R36 91.8 mm to (159.6, 98.8), turned to -90 degrees
- moved C22 91.8 mm to (141.2, 130.4), turned to -90 degrees
- moved R13 91.5 mm to (161.0, 98.4), turned to -90 degrees
- moved R105 90.1 mm to (158.1, 96.2), turned to 180 degrees
- moved C43 90.1 mm to (162.7, 100.8), turned to 90 degrees
- moved C57 89.6 mm to (164.2, 106.0), turned to -90 degrees
- moved C59 89.5 mm to (163.5, 103.1)
- moved C47 88.4 mm to (162.6, 106.0), turned to -90 degrees
- moved R111 86.4 mm to (131.2, 137.0), turned to -90 degrees
- moved C28 86.3 mm to (139.7, 133.3), turned to 0 degrees
- moved R110 85.8 mm to (128.7, 137.0), turned to -90 degrees
- moved U6 85.4 mm to (158.6, 103.2), turned to -90 degrees
- moved R109 85.2 mm to (126.1, 137.0), turned to -90 degrees
- moved R108 85.0 mm to (124.0, 137.0), turned to -90 degrees
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Connections:
- net Net-(J6-PadA4) renamed 5V_USB
- C54 pad 1: GND -> Net-(C53-Pad1)
- C54 pad 2: Net-(C54-Pad2) -> GND
- C56 pad 1: Net-(C56-Pad1) -> Net-(U6-Pad15)
- C57 pad 1: GND -> Net-(U6-Pad15)
- C57 pad 2: Net-(C57-Pad2) -> GND
- C59 pad 1: Net-(C56-Pad1) -> Net-(U6-Pad29)
- C60 pad 1: Net-(C53-Pad1) -> Net-(C60-Pad1)
- J6 pad A1: Net-(J6-PadA1) -> GND
- J6 pad A12: Net-(J6-PadA1) -> GND
- J6 pad A6: unconnected-(J6-PadA6) -> Net-(J6-PadA6)
- J6 pad A7: unconnected-(J6-PadA7) -> Net-(J6-PadA7)
- J6 pad B1: Net-(J6-PadA1) -> GND
- J6 pad B12: Net-(J6-PadA1) -> GND
- J6 pad B6: unconnected-(J6-PadB6) -> Net-(J6-PadA6)
- J6 pad B7: unconnected-(J6-PadB7) -> Net-(J6-PadA7)
- J6 pad S1: unconnected-(J6-PadS1) -> GND
- J7 pad 1: unconnected-(J7-Pad1) -> /SD_DATA1
- J7 pad 2: unconnected-(J7-Pad2) -> /SD_DATA0
- J7 pad 3: unconnected-(J7-Pad3) -> GND
- J7 pad 4: unconnected-(J7-Pad4) -> /SD_CLK
- J7 pad 6: unconnected-(J7-Pad6) -> /SD_CMD
- J7 pad 7: unconnected-(J7-Pad7) -> /SD_DATA3
- J7 pad 8: unconnected-(J7-Pad8) -> /SD_DATA2
- RN1 pad 5: /DRAM_nCS -> /DRAM_ADDR_9
- RN1 pad 6: /DRAM_ODT -> /DRAM_ADDR_13
- RN1 pad 7: /DRAM_nCAS -> /DRAM_ADDR_7
- RN1 pad 8: /DRAM_nRAS -> /DRAM_ADDR_2
- RN2 pad 5: /DRAM_ADDR_3 -> /DRAM_ADDR_6
- RN2 pad 6: /DRAM_ADDR_0 -> /DRAM_ADDR_8
- RN2 pad 7: /DRAM_ADDR_BA2 -> /DRAM_ADDR_14
- RN2 pad 8: /DRAM_ADDR_BA0 -> /DRAM_ADDR_11
- RN4 pad 4: unconnected-(RN4-Pad4) -> GND
- RN4 pad 5: unconnected-(RN4-Pad5) -> /DRAM_ADDR_BA2
- RN4 pad 6: /DRAM_ADDR_7 -> /DRAM_nWE
- RN4 pad 7: /DRAM_ADDR_2 -> /DRAM_nCS
- RN4 pad 8: /DRAM_ADDR_5 -> /DRAM_ODT
- RN5 pad 5: /DRAM_ADDR_14 -> /DRAM_ADDR_BA0
- RN5 pad 6: /DRAM_ADDR_11 -> /DRAM_ADDR_0
- RN5 pad 7: /DRAM_ADDR_9 -> /DRAM_ADDR_15
- RN5 pad 8: /DRAM_ADDR_13 -> /DRAM_ADDR_3
- U1 pad A10: Net-(U1-PadA10) -> /SD_DATA2
- U1 pad A11: Net-(U1-PadA10) -> /USB_SLAVE_CLK
- U1 pad A12: /DRAM_nWE -> /DRAM_ADDR_BA0
- U1 pad A13: /DRAM_ADDR_BA1 -> /DRAM_ADDR_7
- U1 pad A14: /DRAM_ADDR_4 -> /DRAM_ADDR_13
- U1 pad A16: /DRAM_ADDR_14 -> /DRAM_ADDR_5
- U1 pad A17: /DRAM_nRAS -> /DRAM_ADDR_3
- U1 pad A18: /DRAM_ADDR_BA0 -> /DRAM_ADDR_11
- U1 pad A19: /DRAM_nCAS -> /DRAM_nWE
- U1 pad A3: unconnected-(U1-PadA3) -> /USB_HOST_DATA6
- U1 pad A4: unconnected-(U1-PadA4) -> /USB_HOST_DATA4
- U1 pad A5: unconnected-(U1-PadA5) -> /USB_HOST_DATA2
- U1 pad A6: Net-(U1-PadA10) -> /USB_HOST_DATA0
- U1 pad A7: Net-(U1-PadA10) -> /SD_DATA1
- U1 pad A8: Net-(U1-PadA10) -> /SD_DATA0
- U1 pad A9: Net-(U1-PadA10) -> /SD_CMD
- U1 pad B10: Net-(U1-PadA10) -> /USB_SLAVE_DATA3
- U1 pad B11: Net-(U1-PadA10) -> /USB_SLAVE_DATA1
- U1 pad B12: /DRAM_ADDR_15 -> /DRAM_ADDR_BA2
- U1 pad B13: /DRAM_ADDR_1 -> /DRAM_nRESET
- U1 pad B15: /DRAM_ADDR_6 -> /DRAM_ADDR_9
- U1 pad B16: unconnected-(U1-PadB16) -> /DRAM_ADDR_2
- U1 pad B17: unconnected-(U1-PadB17) -> /DRAM_ADDR_0
- U1 pad B19: /DRAM_nCS -> unconnected-(U1-PadB19)
- U1 pad B3: unconnected-(U1-PadB3) -> /USB_HOST_DATA7
- U1 pad B4: unconnected-(U1-PadB4) -> /USB_HOST_DATA5
- U1 pad B5: unconnected-(U1-PadB5) -> /USB_HOST_DATA3
- U1 pad B6: Net-(U1-PadA10) -> /USB_HOST_DATA1
- U1 pad B8: Net-(U1-PadA10) -> /SD_CLK
- U1 pad B9: Net-(U1-PadA10) -> /SD_DATA3
- U1 pad C10: Net-(U1-PadA10) -> /USB_SLAVE_DATA2
- U1 pad C11: Net-(U1-PadA10) -> /USB_SLAVE_DATA0
- U1 pad C12: /DRAM_ADDR_10 -> /DRAM_ADDR_8
- U1 pad C13: unconnected-(U1-PadC13) -> /DRAM_ADDR_1
- U1 pad C14: /DRAM_ADDR_11 -> /DRAM_ADDR_4
- U1 pad C15: /DRAM_ADDR_5 -> /DRAM_ADDR_15
- U1 pad C16: /DRAM_ADDR_8 -> /DRAM_nCAS
- U1 pad C17: /DRAM_ADDR_0 -> /DRAM_ODT
- U1 pad C18: /DRAM_DATA_4 -> unconnected-(U1-PadC18)
- U1 pad C20: unconnected-(U1-PadC20) -> /DRAM_DATA_7
- U1 pad C6: Net-(U1-PadA10) -> /USB_SLAVE_RESET
- U1 pad C7: Net-(U1-PadA10) -> /USB_SLAVE_NXT
- U1 pad C8: Net-(U1-PadA10) -> /USB_SLAVE_CLKOUT
- U1 pad D11: /DRAM_CKE -> /DRAM_ADDR_14
- U1 pad D13: /DRAM_ADDR_3 -> /DRAM_CKE
- U1 pad D14: /DRAM_nRESET -> /DRAM_nCS
- U1 pad D15: /DRAM_ADDR_2 -> /DRAM_nRAS
- U1 pad D16: /DRAM_ADDR_BA2 -> /DRAM_ADDR_10
- U1 pad D17: /DRAM_DATA_6 -> unconnected-(U1-PadD17)
- U1 pad D18: /DRAM_DATA_7 -> unconnected-(U1-PadD18)
- U1 pad D19: unconnected-(U1-PadD19) -> /DRAM_DATA_4
- U1 pad D6: Net-(U1-PadA10) -> unconnected-(U1-PadD6)
- U1 pad D7: Net-(U1-PadA10) -> /USB_SLAVE_DIR
- U1 pad D8: Net-(U1-PadA10) -> /USB_SLAVE_DATA7
- U1 pad D9: Net-(U1-PadA10) -> unconnected-(U1-PadD9)
- U1 pad E11: unconnected-(U1-PadE11) -> /DRAM_ADDR_6
- U1 pad E13: /DRAM_ADDR_13 -> unconnected-(U1-PadE13)
- U1 pad E14: /DRAM_ADDR_7 -> unconnected-(U1-PadE14)
- U1 pad E15: /DRAM_ADDR_9 -> /DRAM_ADDR_BA1
- U1 pad E16: unconnected-(U1-PadE16) -> /DRAM_DATA_14
- U1 pad E17: unconnected-(U1-PadE17) -> /DRAM_DM1
- U1 pad E18: /DRAM_DATA_5 -> /DRAM_DATA_8
- U1 pad E19: /DRAM_DM1 -> unconnected-(U1-PadE19)
- U1 pad E20: unconnected-(U1-PadE20) -> /DRAM_DATA_5
- U1 pad E6: Net-(U1-PadA10) -> /USB_SLAVE_STP
- U1 pad E7: Net-(U1-PadA10) -> /USB_SLAVE_DATA6
- U1 pad E8: Net-(U1-PadA10) -> /USB_SLAVE_DATA5
- U1 pad E9: Net-(U1-PadA10) -> /USB_SLAVE_DATA4
- U1 pad F1: /VGA_B_5 -> /FIFO_WKUP
- U1 pad F16: unconnected-(U1-PadF16) -> /DRAM_DATA_12
- U1 pad F17: /DRAM_DQS0_P -> /DRAM_DQS1_P
- U1 pad F18: unconnected-(U1-PadF18) -> /DRAM_DATA_10
- U1 pad F19: /DRAM_DATA_8 -> /DRAM_DATA_3
- U1 pad F20: /DRAM_DATA_10 -> /DRAM_DATA_1
- U1 pad G1: /VGA_G_5 -> /FIFO_nTXE
- U1 pad G16: /DRAM_DATA_1 -> /DRAM_DATA_9
- U1 pad G18: /DRAM_DQS0_N -> /DRAM_DQS1_N
- U1 pad G19: /DRAM_DQS1_P -> /DRAM_DQS0_P
- U1 pad G2: /VGA_G_4 -> /FIFO_nRXE
- U1 pad G20: unconnected-(U1-PadG20) -> /DRAM_DM0
- U1 pad H1: /VGA_R_5 -> /FIFO_D7
- U1 pad H16: /DRAM_DATA_3 -> /DRAM_DATA_11
- U1 pad H17: /DRAM_DM0 -> unconnected-(U1-PadH17)
- U1 pad H2: /VGA_R_4 -> /FIFO_D6
- U1 pad H20: /DRAM_DQS1_N -> /DRAM_DQS0_N
- U1 pad J1: /VGA_B_3 -> /FIFO_D5
- U1 pad J16: /DRAM_DATA_0 -> /DRAM_DATA_15
- U1 pad J17: /DRAM_DATA_2 -> /DRAM_DATA_13
- U1 pad J18: /DRAM_DATA_13 -> unconnected-(U1-PadJ18)
- U1 pad J19: /DRAM_DATA_9 -> /DRAM_DATA_6
- U1 pad J20: /DRAM_DATA_11 -> /DRAM_DATA_2
- U1 pad J3: /VGA_B_4 -> /FIFO_nWR
- U1 pad J4: unconnected-(U1-PadJ4) -> /FIFO_nRD
- U1 pad J5: unconnected-(U1-PadJ5) -> /VGA_B_5
- U1 pad K1: /VGA_G_3 -> /FIFO_D3
- U1 pad K18: /DRAM_DATA_15 -> unconnected-(U1-PadK18)
- U1 pad K19: /DRAM_DATA_12 -> unconnected-(U1-PadK19)
- U1 pad K2: /VGA_B_2 -> /FIFO_D2
- U1 pad K20: /DRAM_DATA_14 -> /DRAM_DATA_0
- U1 pad K3: unconnected-(U1-PadK3) -> /VGA_B_1
- U1 pad K4: unconnected-(U1-PadK4) -> /VGA_B_3
- U1 pad K5: unconnected-(U1-PadK5) -> /VGA_B_4
- U1 pad L1: /VGA_R_3 -> /FIFO_D1/TX
- U1 pad L16: unconnected-(U1-PadL16) -> /DRAM_DATA_23
- U1 pad L17: /DRAM_DATA_25 -> /DRAM_DATA_17
- U1 pad L18: /DRAM_DATA_26 -> unconnected-(U1-PadL18)
- U1 pad L2: /VGA_R_2 -> /FIFO_D0/RX
- U1 pad L3: /VGA_G_2 -> /FIFO_D4
- U1 pad L4: unconnected-(U1-PadL4) -> /VGA_B_2
- U1 pad L5: unconnected-(U1-PadL5) -> /VGA_G_5
- U1 pad L6: Net-(U1-PadL6) -> +3V3
- U1 pad L7: Net-(U1-PadL6) -> +3V3
- U1 pad M1: /VGA_B_1 -> /VGA_G_0
- U1 pad M17: /DRAM_DQS3_N -> /DRAM_DQS2_N
- U1 pad M18: /DRAM_DATA_30 -> /DRAM_DATA_19
- U1 pad M19: /DRAM_DATA_29 -> unconnected-(U1-PadM19)
- U1 pad M20: /DRAM_DATA_28 -> /DRAM_DM2
- U1 pad M3: unconnected-(U1-PadM3) -> /VGA_G_3
- U1 pad M4: unconnected-(U1-PadM4) -> /VGA_G_4
- U1 pad M6: Net-(U1-PadL6) -> +3V3
- U1 pad N1: /VGA_G_1 -> /VGA_VSYNC
- U1 pad N16: /DRAM_DQS3_P -> /DRAM_DQS2_P
- U1 pad N17: unconnected-(U1-PadN17) -> /DRAM_DATA_16
- U1 pad N18: /DRAM_DATA_31 -> /DRAM_DATA_21
- U1 pad N19: unconnected-(U1-PadN19) -> /DRAM_DATA_26
- U1 pad N2: /VGA_G_0 -> /VGA_HSYNC
- U1 pad N20: unconnected-(U1-PadN20) -> /DRAM_DATA_30
- U1 pad N3: /VGA_B_0 -> /VGA_G_1
- U1 pad N4: unconnected-(U1-PadN4) -> /VGA_G_2
- U1 pad N5: unconnected-(U1-PadN5) -> /VGA_R_0
- U1 pad P1: /VGA_R_1 -> /VGA_R_5
- U1 pad P17: /DRAM_DATA_27 -> /DRAM_DATA_20
- U1 pad P19: /DRAM_DATA_16 -> /DRAM_DATA_28
- U1 pad P2: /VGA_R_0 -> /VGA_R_4
- U1 pad P20: /DRAM_DATA_23 -> /DRAM_DATA_24
- U1 pad P3: /VGA_VSYNC -> /VGA_R_3
- U1 pad P4: /VGA_HSYNC -> /VGA_R_2
- U1 pad P5: unconnected-(U1-PadP5) -> /VGA_R_1
- U1 pad R16: /DRAM_DATA_24 -> /DRAM_DATA_22
- U1 pad R17: /DRAM_DM3 -> /DRAM_DATA_18
- U1 pad R18: /DRAM_DQS2_N -> /DRAM_DQS3_N
- U1 pad R5: unconnected-(U1-PadR5) -> /JTAG_TDI
- U1 pad T17: /DRAM_DM2 -> unconnected-(U1-PadT17)
- U1 pad T18: unconnected-(U1-PadT18) -> /DRAM_DATA_29
- U1 pad T19: /DRAM_DQS2_P -> /DRAM_DQS3_P
- U1 pad T20: /DRAM_DATA_20 -> /DRAM_DATA_31
- U1 pad T5: unconnected-(U1-PadT5) -> /JTAG_TCK
- U1 pad U16: /DRAM_DATA_21 -> unconnected-(U1-PadU16)
- U1 pad U17: /DRAM_DATA_19 -> unconnected-(U1-PadU17)
- U1 pad U18: /DRAM_DATA_17 -> /DRAM_DM3
- U1 pad U19: /DRAM_DATA_22 -> /DRAM_DATA_27
- U1 pad U20: /DRAM_DATA_18 -> /DRAM_DATA_25
- U1 pad U5: unconnected-(U1-PadU5) -> /JTAG_TMS
- U1 pad V4: unconnected-(U1-PadV4) -> /JTAG_TDO
- U10 pad 2: /VGA_R_4 -> unconnected-(U10-Pad2)
- U10 pad 3: /VGA_R_5 -> unconnected-(U10-Pad3)
- U10 pad 4: /VGA_G_4 -> /VGA_B_0
- U10 pad 5: /VGA_G_5 -> /VGA_B_1
- U10 pad 6: /VGA_B_4 -> /VGA_B_2
- U10 pad 7: /VGA_B_5 -> /VGA_B_3
- U10 pad 8: unconnected-(U10-Pad8) -> /VGA_B_4
- U10 pad 9: unconnected-(U10-Pad9) -> /VGA_B_5
- U12 pad 1: unconnected-(U12-Pad1) -> Net-(J6-PadA6)
- U12 pad 2: unconnected-(U12-Pad2) -> Net-(J6-PadA7)
- U12 pad 28: GND -> unconnected-(U12-Pad28)
- U12 pad 7: GND -> unconnected-(U12-Pad7)
- U6 pad 15: Net-(C56-Pad1) -> Net-(U6-Pad15)
- U6 pad 26: Net-(C56-Pad1) -> Net-(U6-Pad15)
- U6 pad 29: Net-(C57-Pad2) -> Net-(U6-Pad29)
- U7 pad 29: Net-(C54-Pad2) -> Net-(C60-Pad1)
- U8 pad 6: /VGA_G_0 -> /VGA_R_2
- U8 pad 7: /VGA_G_1 -> /VGA_R_3
- U8 pad 8: /VGA_B_0 -> /VGA_R_4
- U8 pad 9: /VGA_B_1 -> /VGA_R_5
- U9 pad 2: /VGA_R_2 -> unconnected-(U9-Pad2)
- U9 pad 3: /VGA_R_3 -> unconnected-(U9-Pad3)
- U9 pad 4: /VGA_G_2 -> /VGA_G_0
- U9 pad 5: /VGA_G_3 -> /VGA_G_1
- U9 pad 6: /VGA_B_2 -> /VGA_G_2
- U9 pad 7: /VGA_B_3 -> /VGA_G_3
- U9 pad 8: unconnected-(U9-Pad8) -> /VGA_G_4
- U9 pad 9: unconnected-(U9-Pad9) -> /VGA_G_5
Routing:
- net GND: track 107.3 -> 259.5 mm, vias 27 -> 111
- net DRAM_VREF: track 0.00 -> 97.9 mm, vias 0 -> 8
- net 1V35_DRAM_VCORE: track 8.20 -> 104.8 mm, vias 6 -> 46
- net /DRAM_ADDR_15: track 0.00 -> 90.6 mm, vias 0 -> 4
- net /DRAM_ADDR_12: track 0.00 -> 88.1 mm, vias 0 -> 3
- net /DRAM_ADDR_11: track 0.00 -> 88.0 mm, vias 0 -> 3
- net /DRAM_CKE: track 0.00 -> 85.6 mm, vias 0 -> 3
- net /DRAM_ADDR_0: track 0.00 -> 81.7 mm, vias 0 -> 4
- net /DRAM_ADDR_3: track 0.00 -> 80.5 mm, vias 0 -> 4
- net /DRAM_ADDR_BA2: track 0.00 -> 80.2 mm, vias 0 -> 4
- net /DRAM_nWE: track 0.00 -> 79.0 mm, vias 0 -> 4
- net /DRAM_ADDR_2: track 0.00 -> 77.8 mm, vias 0 -> 4
- net /DRAM_ADDR_9: track 0.00 -> 77.3 mm, vias 0 -> 4
- net /DRAM_ADDR_BA0: track 0.00 -> 77.0 mm, vias 0 -> 3
- net /DRAM_ADDR_13: track 0.00 -> 76.9 mm, vias 0 -> 4
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- added copper zone on F.Cu, net (none)
- added copper zone on B.Cu, net /FPGA_VCORE
- added copper zone on In3.Cu, net /FPGA_VCORE
- added copper zone on In3.Cu, net 1V35_DRAM_VCORE
- added copper zone on B.Cu, net GND
Other:
- board size 100 x 90 mm -> 100 x 90.8 mm
- board text added: "DQ0 routed to: 23mm on F.cu DQ1 routed to: 22mm on F.cu DQ2 routed to: DQ3 routed to: 18mm on F.cu FPGA-U2ADDR routed to: 29.5mm FPGA-U3ADDR routed to:"
- board text added: "SERDES"
- board text removed: "DRAM STACKUP F1.cu V+ In1.Cu -signal In2.Cu - ground In3.Cu - signal In4.Cu - signal B.Cu - ground"

Commit message: merge power
Parts:
- added C100: 22uF, Capacitor_SMD:C_0603_1608Metric, F.Cu at (155.0, 68.7)
- added C101: 22uF, Capacitor_SMD:C_0603_1608Metric, F.Cu at (152.5, 78.8)
- added C102: 22uF, Capacitor_SMD:C_1206_3216Metric, F.Cu at (156.2, 79.6)
- added C103: 22uF, Capacitor_SMD:C_1206_3216Metric, F.Cu at (167.2, 67.8)
- added C104: 22uF, Capacitor_SMD:C_0603_1608Metric, F.Cu at (169.2, 68.6)
- added C105: 22uF, Capacitor_SMD:C_0603_1608Metric, F.Cu at (167.2, 78.9)
- added C106: 22uF, Capacitor_SMD:C_1206_3216Metric, F.Cu at (170.8, 79.6)
- added C68: 0.1uF, Capacitor_SMD:C_0603_1608Metric, F.Cu at (122.2, 19.2)
- added C69: 0.1uF, Capacitor_SMD:C_0603_1608Metric, F.Cu at (110.2, 21.7)
- added C70: 0.1uF, Capacitor_SMD:C_0603_1608Metric, F.Cu at (118.2, 19.2)
- added C71: 0.1uF, Capacitor_SMD:C_0603_1608Metric, F.Cu at (110.2, 29.3)
- added C72: 0.1uF, Capacitor_SMD:C_0603_1608Metric, F.Cu at (122.2, 24.2)
- added C73: 0.1uF, Capacitor_SMD:C_0603_1608Metric, F.Cu at (114.2, 26.8)
- added C74: 0.1uF, Capacitor_SMD:C_0603_1608Metric, F.Cu at (110.2, 19.2)
- added C75: 0.1uF, Capacitor_SMD:C_0603_1608Metric, F.Cu at (114.2, 29.3)
- added C76: 0.1uF, Capacitor_SMD:C_0603_1608Metric, F.Cu at (110.2, 24.2)
- added C77: 0.1uF, Capacitor_SMD:C_0603_1608Metric, F.Cu at (114.2, 21.7)
- added C78: 0.1uF, Capacitor_SMD:C_0603_1608Metric, F.Cu at (114.2, 24.2)
- added C79: 0.1uF, Capacitor_SMD:C_0603_1608Metric, F.Cu at (118.2, 24.2)
- added C80: 0.1uF, Capacitor_SMD:C_0603_1608Metric, F.Cu at (122.2, 21.7)
- added C81: 0.1uF, Capacitor_SMD:C_0603_1608Metric, F.Cu at (118.2, 26.8)
- added C82: 0.1uF, Capacitor_SMD:C_0603_1608Metric, F.Cu at (110.2, 26.8)
- added C83: 0.1uF, Capacitor_SMD:C_0603_1608Metric, F.Cu at (118.2, 21.7)
- added C84: 0.1uF, Capacitor_SMD:C_0603_1608Metric, F.Cu at (126.2, 19.2)
- added C85: 0.1uF, Capacitor_SMD:C_0603_1608Metric, F.Cu at (126.2, 21.7)
- added C86: 0.1uF, Capacitor_SMD:C_0603_1608Metric, F.Cu at (114.2, 19.2)
- added C87: 22uF, Capacitor_SMD:C_1206_3216Metric, F.Cu at (174.4, 67.8)
- added C88: 22uF, Capacitor_SMD:C_0603_1608Metric, F.Cu at (176.4, 68.6)
- added C89: 22uF, Capacitor_SMD:C_0603_1608Metric, F.Cu at (174.4, 78.8)
- added C90: 22uF, Capacitor_SMD:C_1206_3216Metric, F.Cu at (178.1, 79.6)
- added C91: 22uF, Capacitor_SMD:C_1206_3216Metric, F.Cu at (160.1, 67.8)
- added C92: 22uF, Capacitor_SMD:C_0603_1608Metric, F.Cu at (162.1, 68.7)
- added C93: 22uF, Capacitor_SMD:C_0603_1608Metric, F.Cu at (159.9, 78.9)
- added C94: 22uF, Capacitor_SMD:C_1206_3216Metric, F.Cu at (163.5, 79.6)
- added C95: 22uF, Capacitor_SMD:C_1206_3216Metric, F.Cu at (145.6, 67.9)
- added C96: 22uF, Capacitor_SMD:C_0603_1608Metric, F.Cu at (147.6, 68.7)
- added C97: 22uF, Capacitor_SMD:C_0603_1608Metric, F.Cu at (144.9, 78.8)
- added C98: 22uF, Capacitor_SMD:C_1206_3216Metric, F.Cu at (148.5, 79.6)
- added C99: 22uF, Capacitor_SMD:C_1206_3216Metric, F.Cu at (152.9, 67.9)
- added D1: LED, LED_SMD:LED_0603_1608Metric_Pad1.05x0.95mm_HandSolder, F.Cu at (172.9, 80.2)
- added D2: LED, LED_SMD:LED_0603_1608Metric_Pad1.05x0.95mm_HandSolder, F.Cu at (158.3, 80.1)
- added D3: LED, LED_SMD:LED_0603_1608Metric_Pad1.05x0.95mm_HandSolder, F.Cu at (143.3, 80.2)
- added D4: LED, LED_SMD:LED_0603_1608Metric_Pad1.05x0.95mm_HandSolder, F.Cu at (150.7, 80.2)
- added D5: LED, LED_SMD:LED_0603_1608Metric_Pad1.05x0.95mm_HandSolder, F.Cu at (165.7, 80.1)
- added L3: 1uH, Inductor_SMD:L_0805_2012Metric, F.Cu at (173.8, 75.5)
- added L4: 1uH, Inductor_SMD:L_0805_2012Metric, F.Cu at (159.8, 75.5)
- added L5: 1uH, Inductor_SMD:L_0805_2012Metric, F.Cu at (145.1, 75.4)
- added L6: 1uH, Inductor_SMD:L_0805_2012Metric, F.Cu at (152.7, 75.5)
- added L7: 1uH, Inductor_SMD:L_0805_2012Metric, F.Cu at (167.0, 75.5)
- added R1: R220, Resistor_SMD:R_0402_1005Metric_Pad0.72x0.64mm_HandSolder, F.Cu at (121.8, 26.5)
- added R11: 160k, Resistor_SMD:R_0603_1608Metric, F.Cu at (163.5, 71.9)
- added R12: R10, Resistor_SMD:R_0603_1608Metric, F.Cu at (161.5, 78.9)
- added R14: 200k, Resistor_SMD:R_0603_1608Metric, F.Cu at (148.5, 75.6)
- added R15: 160k, Resistor_SMD:R_0603_1608Metric, F.Cu at (148.5, 72.5)
- added R16: R10, Resistor_SMD:R_0603_1608Metric, F.Cu at (146.5, 78.8)
- added R17: 200k, Resistor_SMD:R_0603_1608Metric, F.Cu at (156.2, 75.7)
- added R18: 160k, Resistor_SMD:R_0603_1608Metric, F.Cu at (156.3, 72.0)
- added R19: R10, Resistor_SMD:R_0603_1608Metric, F.Cu at (154.1, 78.8)
- added R21: 200k, Resistor_SMD:R_0603_1608Metric, F.Cu at (170.6, 75.5)
- added R22: 160k, Resistor_SMD:R_0603_1608Metric, F.Cu at (170.6, 72.0)
- added R23: R10, Resistor_SMD:R_0603_1608Metric, F.Cu at (168.8, 78.9)
- added R3: R220, Resistor_SMD:R_0402_1005Metric_Pad0.72x0.64mm_HandSolder, F.Cu at (117.8, 29.0)
- added R4: 200k, Resistor_SMD:R_0603_1608Metric, F.Cu at (177.9, 75.2)
- added R6: 160k, Resistor_SMD:R_0603_1608Metric, F.Cu at (177.9, 72.0)
- added R7: R10, Resistor_SMD:R_0603_1608Metric, F.Cu at (176.1, 78.8)
- added R8: 200k, Resistor_SMD:R_0603_1608Metric, F.Cu at (163.5, 75.7)
- added TP3: TestPoint, TestPoint:TestPoint_Plated_Hole_D2.0mm, F.Cu at (176.1, 63.1)
- added TP4: TestPoint, TestPoint:TestPoint_Plated_Hole_D2.0mm, F.Cu at (161.3, 63.1)
- added TP5: TestPoint, TestPoint:TestPoint_Plated_Hole_D2.0mm, F.Cu at (146.9, 63.1)
- added TP6: TestPoint, TestPoint:TestPoint_Plated_Hole_D2.0mm, F.Cu at (154.2, 63.1)
- added TP7: TestPoint, TestPoint:TestPoint_Plated_Hole_D2.0mm, F.Cu at (168.4, 63.1)
- added U14: AP61300Z6-7, Package_TO_SOT_SMD:SOT-563, F.Cu at (174.3, 71.9)
- added U15: AP61300Z6-7, Package_TO_SOT_SMD:SOT-563, F.Cu at (160.0, 71.9)
- added U16: AP61300Z6-7, Package_TO_SOT_SMD:SOT-563, F.Cu at (145.6, 71.9)
- added U17: AP61300Z6-7, Package_TO_SOT_SMD:SOT-563, F.Cu at (152.9, 71.9)
- added U18: AP61300Z6-7, Package_TO_SOT_SMD:SOT-563, F.Cu at (167.2, 71.9)
- added kibuzzard-620E4897: G***, kibuzzard-620E4897, F.Cu at (143.5, 64.8)
- added kibuzzard-620E48A0: G***, kibuzzard-620E48A0, F.Cu at (150.8, 64.8)
- added kibuzzard-620E48AE: G***, kibuzzard-620E48AE, F.Cu at (157.7, 65.1)
- added kibuzzard-620E48DF: G***, kibuzzard-620E48DF, F.Cu at (172.8, 64.8)
- added kibuzzard-620E48DF: G***, kibuzzard-620E48DF, F.Cu at (165.2, 64.8)
- moved U12 2.15 mm to (184.7, 69.5)
- moved U11 1.20 mm to (125.1, 107.1)
- moved J5 0.73 mm to (104.7, 107.7)
Connections:
- J5 pad L1: unconnected-(J5-PadL1) -> Net-(J5-PadL1)
- J5 pad L2: unconnected-(J5-PadL2) -> Net-(J5-PadL2)
- J5 pad L3: unconnected-(J5-PadL3) -> Net-(J5-PadL3)
- J5 pad L4: unconnected-(J5-PadL4) -> Net-(J5-PadL4)
- J5 pad S1: Net-(J5-PadS1) -> GND
- J5 pad S2: Net-(J5-PadS1) -> GND
- U11 pad 12: unconnected-(U11-Pad12) -> +1V2
- U11 pad 13: unconnected-(U11-Pad13) -> +1V2
- U11 pad 16: unconnected-(U11-Pad16) -> +3V3
- U11 pad 19: unconnected-(U11-Pad19) -> Net-(J5-PadL2)
- U11 pad 20: unconnected-(U11-Pad20) -> +3V3
- U11 pad 21: unconnected-(U11-Pad21) -> Net-(J5-PadL4)
- U11 pad 22: unconnected-(U11-Pad22) -> +1V2
- U11 pad 24: unconnected-(U11-Pad24) -> /TX0
- U11 pad 25: unconnected-(U11-Pad25) -> /TX1
- U11 pad 26: unconnected-(U11-Pad26) -> /TX2
- U11 pad 27: unconnected-(U11-Pad27) -> /TX3
- U11 pad 29: unconnected-(U11-Pad29) -> +1V2
- U11 pad 30: unconnected-(U11-Pad30) -> +3V3
- U11 pad 32: unconnected-(U11-Pad32) -> /TX_CLK
- U11 pad 33: unconnected-(U11-Pad33) -> /TX_CTRL
- U11 pad 35: unconnected-(U11-Pad35) -> +1V2
- U11 pad 36: unconnected-(U11-Pad36) -> /RX3
- U11 pad 37: unconnected-(U11-Pad37) -> +3V3
- U11 pad 38: unconnected-(U11-Pad38) -> /RX2
- U11 pad 4: unconnected-(U11-Pad4) -> +1V2
- U11 pad 40: unconnected-(U11-Pad40) -> +1V2
- U11 pad 41: unconnected-(U11-Pad41) -> /RX1
- U11 pad 42: unconnected-(U11-Pad42) -> /RX0
- U11 pad 43: unconnected-(U11-Pad43) -> /RX_CTRL
- U11 pad 44: unconnected-(U11-Pad44) -> +3V3
- U11 pad 46: unconnected-(U11-Pad46) -> /RX_CLK
- U11 pad 48: unconnected-(U11-Pad48) -> /MDC
- U11 pad 49: unconnected-(U11-Pad49) -> /MDIO
- U11 pad 5: unconnected-(U11-Pad5) -> +1V2
- U11 pad 51: unconnected-(U11-Pad51) -> /INT
- U11 pad 52: unconnected-(U11-Pad52) -> +1V2
- U11 pad 54: unconnected-(U11-Pad54) -> +1V2
- U11 pad 55: unconnected-(U11-Pad55) -> /CLK125
- U11 pad 56: unconnected-(U11-Pad56) -> /RESET
- U11 pad 58: unconnected-(U11-Pad58) -> +1V2
- U11 pad 6: unconnected-(U11-Pad6) -> +3V3
- U11 pad 61: unconnected-(U11-Pad61) -> +3V3
- U11 pad 64: unconnected-(U11-Pad64) -> +3V3
Routing:
- net +5V: track 0.00 -> 11.4 mm, vias 0 -> 18
- net Net-(R17-Pad2): track 0.00 -> 6.86 mm
- net Net-(R11-Pad1): track 0.00 -> 6.84 mm
- net Net-(R21-Pad2): track 0.00 -> 6.55 mm
- net GND: track 259.5 -> 265.8 mm, vias 111 -> 221
- net Net-(R4-Pad2): track 0.00 -> 6.26 mm
- net Net-(R14-Pad2): track 0.00 -> 5.95 mm
- net Net-(D4-Pad2): track 0.00 -> 4.29 mm
- net /1V2: track 0.00 -> 4.02 mm
- net /1V2_FPGA: track 0.00 -> 3.88 mm, vias 0 -> 10
- net /1V35: track 0.00 -> 3.83 mm, vias 0 -> 10
- net Net-(D3-Pad2): track 0.00 -> 3.72 mm
- net Net-(D1-Pad2): track 0.00 -> 3.65 mm
- net Net-(D5-Pad2): track 0.00 -> 3.61 mm
- net /2V5: track 0.00 -> 3.58 mm, vias 0 -> 10
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- added copper zone on F.Cu, net +5V
- added copper zone on F.Cu, net /1V2
- added copper zone on F.Cu, net /1V2_FPGA
- added copper zone on F.Cu, net /1V35
- added copper zone on F.Cu, net /2V5
- added copper zone on F.Cu, net /3V3
- added copper zone on F.Cu, net GND
- added copper zone on F.Cu, net Net-(L3-Pad1)
- added copper zone on F.Cu, net Net-(L4-Pad1)
- added copper zone on F.Cu, net Net-(L5-Pad1)
- added copper zone on F.Cu, net Net-(L6-Pad1)
- added copper zone on F.Cu, net Net-(L7-Pad1)
